File: Gov_TrkU/Gov_Tracker.kicad_pcb (KiCad board)
At the start: 2 copper layers, 320 x 136 mm, 684 parts, among them CN1 Main_Connector, CN2 Main_Connector, CN3 Main_Connector, CN4 Main_Connector, J1 Conn_01x02, J10 Prog_T, J11 Debug, J12 USB_B_Mini, J13 USB_Con, J14 ANT, J15 Conn_Coaxial, J16 Debug/GPS_DBG, J17 Conn_Coaxial, J18 Prog_G, J19 Prog_T, J2 USB_B_Mini, J20 Debug, J21 Conn_01x02, J22 USB_B_Mini, J23 USB_Con, J24 ANT, J25 Conn_Coaxial, J26 Debug/GPS_DBG, J27 Conn_Coaxial, J28 Prog_G, J29 Prog_T, J3 USB_Con, J30 Debug, J31 Conn_01x02, J32 USB_B_Mini, J33 USB_Con, J34 ANT, J35 Conn_Coaxial, J36 Debug/GPS_DBG, J37 Conn_Coaxial, J38 Prog_G, J39 Prog_T, J4 ANT, J40 Debug, J5 Conn_Coaxial, J6 Debug/GPS_DBG, J7 Conn_Coaxial, J8 Conn_01x02, J9 Prog_G, K2 G5Q-1, K3 SRA-05VDC-CL, K4 G5Q-1, K5 SRA-05VDC-CL, K6 G5Q-1, K7 SRA-05VDC-CL, K8 G5Q-1, K9 SRA-05VDC-CL, Q1 SI2333DS, Q10 BC817, Q11 SI2333DS, Q12 BC817, Q13 BC817, Q14 BSS84, Q15 BC817, Q16 SI2333DS, Q17 BC817, Q18 BC817, Q19 BSS84, Q2 BC817, Q20 BC817, Q3 BC817, Q4 BSS84, Q5 BC817, Q6 SI2333DS, Q7 BC817, Q8 BC817, Q9 BSS84, U10 LM2596S-5, U11 LM393, U12 W25Q128JVS, U13 STM32F103RCTx, U14 NEO-6M-GPS, U15 SY7208B, U16 LM1117-3.3, U17 MCP73831-5-OT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

Commit message: Made amendments
Parts:
- removed ? (x9): , 
- removed BT2, BT3, BT4: 1056, 1056:BAT_1056
- removed BZ2, BZ3, BZ4: Buzzer, Buzzer_Beeper:MagneticBuzzer_ProSignal_ABI-009-RC
- removed C100, C101, C146, C147, C54, C55: 10uF/25V, Capacitor_THT:CP_Radial_D5.0mm_P2.50mm
- removed C102, C148, C56: 1uF/16V, Capacitor_SMD:C_0603_1608Metric
- removed C103, C149, C57: 0.1uF/16V, Capacitor_SMD:C_0603_1608Metric
- removed C104, C150, C58: 100uFx6.3v, Capacitor_SMD:C_Elec_5x5.8
- removed C105, C151, C59: 220uF/10v, Capacitor_SMD:CP_Elec_8x6.5
- removed C106, C118, C152, C164, C60, C72: 0.1uFx/10V, Capacitor_SMD:C_0805_2012Metric
- removed C107, C138, C142, C143, C153, C184, C50, C51, C61, C92, C96, C97: 1uF, Capacitor_SMD:C_0603_1608Metric
- removed C108, C109, C132, C133, C154, C155, C178, C179, C62, C63, C86, C87: 18pF, Capacitor_SMD:C_0603_1608Metric
- removed C110, C112, C114, C116, C119, C121, C134, C136, C156, C158, C160, C162, C165, C167, C180, C182, C64, C66, C68, C70, C73, C75, C88, C90: 1uF/6.3V, Capacitor_SMD:C_0603_1608Metric
- removed C111, C113, C115, C117, C120, C122, C135, C137, C157, C159, C161, C163, C166, C168, C181, C183, C65, C67, C69, C71, C74, C76, C89, C91: 0.1uF/6.3V, Capacitor_SMD:C_0603_1608Metric
- removed C123, C124, C125, C126, C127, C169, C170, C171, C172, C173, C77, C78, C79, C80, C81: 0.1uF, Capacitor_SMD:C_0603_1608Metric
- removed C128, C131, C174, C177, C82, C85: 22pF, Capacitor_SMD:C_0603_1608Metric
- removed C129, C175, C83: 330uF, Capacitor_Tantalum_SMD:CP_EIA-6032-15_Kemet-U
- removed C130, C176, C84: 10uFx/10V, Capacitor_SMD:C_0603_1608Metric
- removed C139, C141, C3, C49, C93, C95: 220uF/25V, Capacitor_SMD:CP_Elec_8x6.9
- removed C140, C48, C94: 10uFx16v, Capacitor_SMD:C_0603_1608Metric
- removed C144, C145, C52, C53, C98, C99: 10uF/16V, Capacitor_SMD:C_0603_1608Metric
- removed CN2, CN3, CN4: Main_Connector, 66201821122:66201821122
- removed D24, D33, D34, D38, D44, D45, D47, D56, D57, D61, D67, D68, D70, D79, D80, D84, D90, D91: 3.9 Zener, Diode_SMD:D_SOD-123
- removed D25, D26, D28, D30, D48, D49, D51, D53, D71, D72, D74, D76: Schottkey/1A, Diode_SMD:D_SMA
- removed D27, D50, D73: R_LED, LED_SMD:LED_0805_2012Metric
- removed D29, D52, D75: G_LED, LED_SMD:LED_0805_2012Metric
- removed D31, D54, D77: GPRS_LED, LED_SMD:LED_0805_2012Metric
- removed D32, D43, D55, D66, D78, D89: G_Purpose, Diode_SMD:D_SMA
- removed D35, D58, D81: PW_LED, LED_SMD:LED_0805_2012Metric
- removed D36, D59, D82: Power, LED_SMD:LED_0805_2012Metric
- removed D37, D60, D83: Schottkey, Diode_SMD:D_SOD-123
- removed D39, D62, D85: G_purpose, Diode_SMD:D_SMA
- removed D40, D63, D86: ST, LED_SMD:LED_0805_2012Metric
- removed D41, D64, D87: NW, LED_SMD:LED_0805_2012Metric
- removed D42, D65, D88: 1N4148, Diode_SMD:D_SOD-123
- removed D46, D69, D92: ?, Diode_SMD:D_SMA
- removed F2, F3, F4: 30V/0.09A, Fuse:Fuse_BelFuse_0ZRE0005FF_L8.3mm_W3.8mm
- removed FID10, FID16, FID22: Fiducial, Fiducial:Fiducial_1.5mm_Mask3mm
- removed FID11, FID12, FID17, FID18, FID23, FID24: Fiducial, Fiducial:Fiducial_0.75mm_Mask1.5mm
- removed FID13, FID14, FID15, FID19, FID20, FID21, FID7, FID8, FID9: Fiducial, Fiducial:Fiducial_1mm_Mask3mm
- removed J12, J22, J32: USB_B_Mini, Connector_USB:USB_Mini-B_Lumberg_2486_01_Horizontal
- removed J13, J23, J33: USB_Con, Connector_PinSocket_2.54mm:PinSocket_1x04_P2.54mm_Vertical
- removed J14, J24, J34: ANT, Connector_Coaxial:SMA_Amphenol_132291_Vertical
- removed J15, J25, J35: Conn_Coaxial, Connector_Coaxial:SMA_Amphenol_132291_Vertical
- removed J16, J26, J36: Debug/GPS_DBG, Connector_PinSocket_2.54mm:PinSocket_1x05_P2.54mm_Vertical
- removed J17, J27, J37: Conn_Coaxial, Connector_Coaxial:U.FL_Molex_MCRF_73412-0110_Vertical
- removed J18, J28, J38: Prog_G, Connector_PinSocket_2.54mm:PinSocket_1x06_P2.54mm_Vertical
- removed J19, J29, J39: Prog_T, Connector_PinSocket_2.54mm:PinSocket_1x06_P2.54mm_Vertical
- removed J20, J30, J40: Debug, Connector_PinHeader_2.54mm:PinHeader_1x03_P2.54mm_Vertical
- removed J21, J31, J8: Conn_01x02, Connector_JST:JST_PH_B2B-PH-K_1x02_P2.00mm_Vertical
- removed JP2, JP3, JP4: Analog fuel jumper, Jumper:SolderJumper-2_P1.3mm_Open_RoundedPad1.0x1.5mm
- removed K4, K6, K8: G5Q-1, Relay_THT:Relay_SPDT_Omron-G5LE-1
- removed K5, K7, K9: SRA-05VDC-CL, SRA-05VDC-CL:RELAY_SRA-05VDC-CL
- removed L10, L3, L7: L-US, Inductor_SMD:L_Taiyo-Yuden_NR-60xx
- removed L11, L4, L8: INDUCTOR, Inductor_SMD:L_Pulse_PA4320
- removed L12, L6, L9: 22nH, Inductor_SMD:L_1206_3216Metric
- removed Q10, Q12, Q13, Q15, Q17, Q18, Q20, Q7, Q8: BC817, Package_TO_SOT_SMD:SOT-23
- removed Q11, Q16, Q6: SI2333DS, Package_TO_SOT_SMD:SC-59
- removed Q14, Q19, Q9: BSS84, Package_TO_SOT_SMD:SOT-23
- removed R100, R126, R145, R150, R176, R195, R200, R76, R95: 100k, Resistor_SMD:R_0603_1608Metric
- removed R101, R105, R106, R107, R114, R116, R121, R125, R127, R139, R148, R149, R151, R155, R156, R157, R164, R166, R171, R175, R177, R189, R198, R199, R201, R55, R56, R57, R64, R66, R71, R75, R77, R89, R98, R99: 1k, Resistor_SMD:R_0603_1608Metric
- removed R102, R152, R202: 22, Resistor_SMD:R_0603_1608Metric
- removed R103, R104, R111, R113, R120, R122, R123, R124, R128, R129, R130, R131, R133, R136, R143, R144, R146, R153, R154, R161, R163, R170, R172, R173, R174, R178, R179, R180, R181, R183, R186, R193, R194, R196, R46, R48, R61, R63, R70, R72, R73, R74, R78, R79, R80, R81, R83, R86, R93, R94, R96: 10k, Resistor_SMD:R_0603_1608Metric
- removed R108, R158, R58: 8.2k, Resistor_SMD:R_0603_1608Metric
- removed R109, R159, R59: 1.1k, Resistor_SMD:R_0603_1608Metric
- removed R110, R112, R160, R162, R60, R62: 33k, Resistor_SMD:R_0603_1608Metric
- removed R115, R165, R65: 5.1k, Resistor_SMD:R_0603_1608Metric
- removed R117, R167, R67: 2k, Resistor_SMD:R_0603_1608Metric
- removed R118, R119, R168, R169, R68, R69: 33, Resistor_SMD:R_0603_1608Metric
- removed R132, R137, R138, R140, R141, R142, R182, R187, R188, R190, R191, R192, R82, R87, R88, R90, R91, R92: 10K, Resistor_SMD:R_0603_1608Metric
- removed R134, R135, R184, R185, R84, R85: 1K(1%)0.1W, Resistor_SMD:R_0603_1608Metric
- removed R147, R197, R97: 3.3k, Resistor_SMD:R_0603_1608Metric
- removed REF**: MountingHole_2.7mm, MountingHole:MountingHole_2.7mm
- removed REF** (x2): Fiducial_0.75mm_Mask1.5mm, Fiducial:Fiducial_0.75mm_Mask1.5mm
- removed TP10, TP13, TP7: BT, TestPoint:TestPoint_Pad_1.0x1.0mm
- removed TP11, TP5, TP8: 5V, TestPoint:TestPoint_Pad_1.0x1.0mm
- removed TP12, TP6, TP9: 3.3V, TestPoint:TestPoint_Pad_1.0x1.0mm
- removed U10, U26, U38: LM2596S-5, Package_TO_SOT_SMD:TO-263-5_TabPin3
- removed U15, U27, U39: SY7208B, Package_TO_SOT_SMD:SOT-23-6
- removed U16, U28, U40: LM1117-3.3, Package_TO_SOT_SMD:SOT-223-3_TabPin2
- removed U17, U29, U41: MCP73831-5-OT, Package_TO_SOT_SMD:SOT-23-5
- removed U18, U24, U30, U36, U42, U48: STM32F103RCTx, Package_QFP:LQFP-64_10x10mm_P0.5mm
- removed U19, U31, U43: 693021020811, simcard:693021020811
- removed U20, U32, U44: SIM800C, RF_GSM:SIMCom_SIM800C
- removed U21, U33, U45: MAX3232, MAX3232EUE:SOP65P640X110-16N
- removed U22, U34, U46: LM393, LM393:SO08
- removed U23, U35, U47: W25Q128JVS, Package_SO:SOIC-8_5.23x5.23mm_P1.27mm
- removed U25, U37, U49: NEO-6M-GPS, NEO-6M-GPS:XCVR_NEO-6M-GPS
- removed Y10, Y12, Y2, Y3, Y7, Y9: 8MHz, Crystal:Crystal_HC49-U_Vertical
- removed Y11, Y6, Y8: 32.678kHz, Crystal:Crystal_DS10_D1.0mm_L4.3mm_Vertical
- moved J4 100.4 mm to (176.2, 132.3)
- moved BT1 100.4 mm to (166.3, 65.5)
- moved C14 100.4 mm to (151.4, 115.2)
- moved C22 100.4 mm to (148.8, 60.6)
- moved C24 100.4 mm to (142.3, 77.6)
- moved C28 100.4 mm to (166.1, 72.5)
- moved C30 100.4 mm to (186.8, 70.3)
- moved C34 100.4 mm to (149.6, 107.7)
- moved C38 100.4 mm to (158.4, 116.0)
- moved C42 100.4 mm to (158.3, 81.5)
- moved C5 100.4 mm to (141.3, 80.3)
- moved CN1 100.4 mm to (146.9, 131.6)
- moved D14 100.4 mm to (190.9, 121.0)
- moved D23 100.4 mm to (138.9, 113.8)
- moved D8 100.4 mm to (129.1, 65.2)
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Routing:
- net GND: track 4014.9 -> 1006.3 mm, vias 280 -> 71
- net +3V3: track 1501.1 -> 375.3 mm, vias 36 -> 9
- net 5L: track 886.3 -> 221.6 mm, vias 24 -> 6
- net +5V: track 794.8 -> 198.7 mm, vias 24 -> 6
- net D-: track 496.1 -> 124.0 mm, vias 4 -> 1
- net D+: track 490.7 -> 122.7 mm, vias 4 -> 1
- net IGNITION_KEY: track 468.8 -> 117.2 mm, vias 20 -> 5
- net DOOR1: track 466.4 -> 116.6 mm, vias 8 -> 2
- net GOV_LD_PIN: track 451.8 -> 113.0 mm, vias 4 -> 1
- net TRACKER_LED: track 439.4 -> 109.9 mm, vias 12 -> 3
- net REC_LD_PIN: track 394.8 -> 98.7 mm, vias 8 -> 2
- net RELAY: track 375.7 -> 93.9 mm, vias 16 -> 4
- net FUEL_TX: track 352.0 -> 88.0 mm, vias 28 -> 7
- net PRNT_BTN: track 350.9 -> 87.7 mm, vias 12 -> 3
- net PROG_BUTTON: track 305.8 -> 76.4 mm, vias 4 -> 1
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- removed copper zone on B.Cu, net (none)
- removed copper zone on F.Cu, net (none)
Other:
- board size 320 x 136 mm -> 75 x 91 mm
- board text added: "Gov_Trk 5.2.5 sim800"
- board text removed: "v-cut"
