File: Gov_TrkU_panel/Gov_tracker_Panel/Gov_tracker_Panel.kicad_pcb (KiCad board)
At the start: 2 copper layers, 320 x 255 mm, 685 parts, among them CN1 Main_Connector, J1 Conn_01x02, J10 Prog_T, J11 Debug, J2 USB_B_Mini, J3 USB_Con, J4 ANT, J5 Conn_Coaxial, J6 Debug/GPS_DBG, J7 Conn_Coaxial, J9 Prog_G, K2 G5Q-1, K3 SRA-05VDC-CL, Q1 SI2333DS, Q2 BC817, Q3 BC817, Q4 BSS84, Q5 BC817, U11 LM393, U12 W25Q128JVS, U13 STM32F103RCTx, U14 NEO-6M-GPS, U2 LM2596S-5, U3 SY7208B, U4 LM1117-3.3, U5 MCP73831-5-OT, U6 STM32F103RCTx, U7 693021020811, U8 SIM800C, U9 MAX3232, Y1 8MHz, Y4 32.678kHz, Y5 8MHz

Commit message: Panel almost complete
Parts:
- removed the BT1 at (684.3, 466.5)
- removed the BT1 at (609.3, 466.5)
- removed the BT1 at (834.3, 466.5)
- removed the BT1 at (759.3, 466.5)
- removed the BZ1 at (688.4, 464.8)
- removed the BZ1 at (613.4, 464.8)
- removed the BZ1 at (763.4, 464.8)
- removed the BZ1 at (838.4, 464.8)
- removed the C1 at (810.7, 505.1)
- removed the C1 at (660.7, 505.1)
- removed the C1 at (735.7, 505.1)
- removed the C1 at (585.7, 505.1)
- removed the C10 at (801.8, 478.0)
- removed the C10 at (651.8, 478.0)
- removed the C10 at (576.8, 478.0)
- removed the C10 at (726.8, 478.0)
- removed the C11 at (652.5, 481.1)
- removed the C11 at (802.5, 481.1)
- removed the C11 at (577.5, 481.1)
- removed the C11 at (727.5, 481.1)
- removed the C12 at (779.6, 493.8)
- removed the C12 at (629.6, 493.8)
- removed the C12 at (854.6, 493.8)
- removed the C12 at (704.6, 493.8)
- removed the C13 at (599.3, 524.8)
- removed the C13 at (749.3, 524.8)
- removed the C13 at (674.3, 524.8)
- removed the C13 at (824.3, 524.8)
- removed the C14 at (744.4, 516.2)
- removed the C14 at (669.4, 516.2)
- removed the C14 at (819.4, 516.2)
- removed the C14 at (594.4, 516.2)
- removed the C15 at (595.0, 507.4)
- removed the C15 at (670.0, 507.4)
- removed the C15 at (745.0, 507.4)
- removed the C15 at (820.0, 507.4)
- removed the C16 at (683.9, 486.2)
- removed the C16 at (608.9, 486.2)
- removed the C16 at (758.9, 486.2)
- removed the C16 at (833.9, 486.2)
- removed the C17 at (611.6, 481.6)
- removed the C17 at (686.6, 481.6)
- removed the C17 at (761.6, 481.6)
- removed the C17 at (836.6, 481.6)
- removed the C18 at (764.7, 481.6)
- removed the C18 at (614.7, 481.6)
- removed the C18 at (839.7, 481.6)
- removed the C18 at (689.7, 481.6)
- removed the C19 at (825.9, 461.9)
- removed the C19 at (675.9, 461.9)
- removed the C19 at (750.9, 461.9)
- removed the C19 at (600.9, 461.9)
- removed the C2 at (702.5, 506.4)
- removed the C2 at (852.5, 506.4)
- removed the C2 at (627.5, 506.4)
- removed the C2 at (777.5, 506.4)
- removed the C20 at (825.9, 463.7)
- removed the C20 at (675.9, 463.7)
- removed the C20 at (600.9, 463.7)
- removed the C20 at (750.9, 463.7)
- removed the C21 at (591.9, 463.6)
- removed the C21 at (666.9, 463.6)
- removed the C21 at (741.9, 463.6)
- removed the C21 at (816.9, 463.6)
- removed the C22 at (816.8, 461.6)
- removed the C22 at (741.8, 461.6)
- removed the C22 at (666.8, 461.6)
- removed the C22 at (591.8, 461.6)
- removed the C23 at (661.1, 482.5)
- removed the C23 at (736.1, 482.5)
- removed the C23 at (586.1, 482.5)
- removed the C23 at (811.1, 482.5)
- removed the C24 at (585.3, 478.6)
- removed the C24 at (660.3, 478.6)
- removed the C24 at (735.3, 478.6)
- removed the C24 at (810.3, 478.6)
- removed the C25 at (829.7, 477.6)
- removed the C25 at (604.7, 477.6)
- removed the C25 at (754.7, 477.6)
- removed the C25 at (679.7, 477.6)
- removed the C26 at (831.6, 477.7)
- removed the C26 at (606.6, 477.7)
- removed the C26 at (681.6, 477.7)
- removed the C26 at (756.6, 477.7)
- removed the C27 at (825.5, 510.0)
- removed the C27 at (675.5, 510.0)
- removed the C27 at (750.5, 510.0)
- removed the C27 at (600.5, 510.0)
- removed the C28 at (684.0, 473.6)
- removed the C28 at (834.0, 473.6)
- removed the C28 at (759.0, 473.6)
- removed the C28 at (609.0, 473.6)
- removed the C29 at (760.7, 473.6)
- removed the C29 at (610.7, 473.6)
- removed the C29 at (685.7, 473.6)
- removed the C29 at (835.7, 473.6)
- removed the C30 at (704.8, 471.3)
- removed the C30 at (779.8, 471.3)
- removed the C30 at (629.8, 471.3)
- removed the C30 at (854.8, 471.3)
- removed the C31 at (857.0, 471.3)
- removed the C31 at (782.0, 471.3)
- removed the C31 at (632.0, 471.3)
- removed the C31 at (707.0, 471.3)
- removed the C32 at (810.5, 499.1)
- removed the C32 at (735.5, 499.1)
- removed the C32 at (585.5, 499.1)
- removed the C32 at (660.5, 499.1)
- removed the C33 at (670.3, 507.9)
- removed the C33 at (745.3, 507.9)
- removed the C33 at (820.3, 507.9)
- removed the C33 at (595.3, 507.9)
- removed the C34 at (667.5, 508.6)
- removed the C34 at (592.5, 508.6)
- removed the C34 at (817.5, 508.6)
- removed the C34 at (742.5, 508.6)
- removed the C35 at (739.0, 499.1)
- removed the C35 at (814.0, 499.1)
- removed the C35 at (589.0, 499.1)
- removed the C35 at (664.0, 499.1)
- removed the C36 at (814.0, 497.1)
- removed the C36 at (589.0, 497.1)
- removed the C36 at (739.0, 497.1)
- removed the C36 at (664.0, 497.1)
- removed the C37 at (743.4, 485.0)
- removed the C37 at (593.4, 485.0)
- removed the C37 at (668.4, 485.0)
- removed the C37 at (818.4, 485.0)
- removed the C38 at (676.4, 517.0)
- removed the C38 at (751.4, 517.0)
- removed the C38 at (601.4, 517.0)
- removed the C38 at (826.4, 517.0)
- removed the C39 at (600.6, 507.1)
- removed the C39 at (675.6, 507.1)
- removed the C39 at (750.6, 507.1)
- removed the C39 at (825.6, 507.1)
- removed the C4 at (569.9, 485.6)
- removed the C4 at (794.9, 485.6)
- removed the C4 at (644.9, 485.6)
- removed the C4 at (719.9, 485.6)
- removed the C40 at (743.4, 483.5)
- removed the C40 at (668.4, 483.5)
- removed the C40 at (818.4, 483.5)
- removed the C40 at (593.4, 483.5)
- removed the C41 at (673.3, 482.4)
- removed the C41 at (598.3, 482.4)
- removed the C41 at (748.3, 482.4)
- removed the C41 at (823.3, 482.4)
- removed the C42 at (826.3, 482.5)
- removed the C42 at (751.3, 482.5)
- removed the C42 at (601.3, 482.5)
- removed the C42 at (676.3, 482.5)
- removed the C43 at (776.1, 489.2)
- removed the C43 at (851.1, 489.2)
- removed the C43 at (701.1, 489.2)
- removed the C43 at (626.1, 489.2)
- removed the C44 at (853.8, 489.2)
- removed the C44 at (628.8, 489.2)
- removed the C44 at (703.8, 489.2)
- removed the C44 at (778.8, 489.2)
- removed the C45 at (610.0, 477.8)
- removed the C45 at (685.0, 477.8)
- removed the C45 at (835.0, 477.8)
- removed the C45 at (760.0, 477.8)
- removed the C46 at (834.9, 479.7)
- removed the C46 at (609.9, 479.7)
- removed the C46 at (684.9, 479.7)
- removed the C46 at (759.9, 479.7)
- removed the C47 at (745.1, 504.4)
- removed the C47 at (670.1, 504.4)
- removed the C47 at (820.1, 504.4)
- removed the C47 at (595.1, 504.4)
- removed the C5 at (734.3, 481.3)
- removed the C5 at (659.3, 481.3)
- removed the C5 at (809.3, 481.3)
- removed the C5 at (584.3, 481.3)
- removed the C6 at (579.0, 491.0)
- removed the C6 at (804.0, 491.0)
- removed the C6 at (654.0, 491.0)
- removed the C6 at (729.0, 491.0)
- removed the C7 at (781.3, 501.4)
- removed the C7 at (631.3, 501.4)
- removed the C7 at (706.3, 501.4)
- removed the C7 at (856.3, 501.4)
- removed the C8 at (707.0, 505.0)
- removed the C8 at (632.0, 505.0)
- removed the C8 at (857.0, 505.0)
- removed the C8 at (782.0, 505.0)
- removed the C9 at (578.7, 484.0)
- removed the C9 at (653.7, 484.0)
- removed the C9 at (803.7, 484.0)
- removed the C9 at (728.7, 484.0)
- removed the CN1 at (664.9, 532.6)
- removed the CN1 at (814.9, 532.6)
- removed the CN1 at (739.9, 532.6)
- removed the CN1 at (589.9, 532.6)
- removed the D1 at (586.7, 520.4)
- removed the D1 at (811.7, 520.4)
- removed the D1 at (661.7, 520.4)
- removed the D1 at (736.7, 520.4)
- removed the D10 at (695.0, 473.5)
- removed the D10 at (620.0, 473.5)
- removed the D10 at (845.0, 473.5)
- removed the D10 at (770.0, 473.5)
- removed the D11 at (701.1, 470.3)
- removed the D11 at (776.1, 470.3)
- removed the D11 at (851.1, 470.3)
- removed the D11 at (626.1, 470.3)
- removed the D12 at (717.1, 470.4)
- removed the D12 at (567.1, 470.4)
- removed the D12 at (642.1, 470.4)
- removed the D12 at (792.1, 470.4)
- removed the D13 at (768.9, 498.2)
- removed the D13 at (618.9, 498.2)
- removed the D13 at (843.9, 498.2)
- removed the D13 at (693.9, 498.2)
- removed the D14 at (633.9, 522.0)
- removed the D14 at (858.9, 522.0)
- removed the D14 at (783.9, 522.0)
- removed the D14 at (708.9, 522.0)
- removed the D15 at (737.8, 463.2)
- removed the D15 at (587.8, 463.2)
- removed the D15 at (662.8, 463.2)
- removed the D15 at (812.8, 463.2)
- removed the D16 at (825.4, 504.7)
- removed the D16 at (600.4, 504.7)
- removed the D16 at (750.4, 504.7)
- removed the D16 at (675.4, 504.7)
- removed the D17 at (705.8, 515.4)
- removed the D17 at (630.8, 515.4)
- removed the D17 at (855.8, 515.4)
- removed the D17 at (780.8, 515.4)
- removed the D18 at (630.7, 512.3)
- removed the D18 at (855.7, 512.3)
- removed the D18 at (705.7, 512.3)
- removed the D18 at (780.7, 512.3)
- removed the D19 at (658.9, 481.9)
- removed the D19 at (733.9, 481.9)
- removed the D19 at (808.9, 481.9)
- removed the D19 at (583.9, 481.9)
- removed the D2 at (797.3, 504.5)
- removed the D2 at (722.3, 504.5)
- removed the D2 at (647.3, 504.5)
- removed the D2 at (572.3, 504.5)
- removed the D20 at (663.5, 524.4)
- removed the D20 at (738.5, 524.4)
- removed the D20 at (588.5, 524.4)
- removed the D20 at (813.5, 524.4)
- removed the D21 at (827.5, 492.0)
- removed the D21 at (602.5, 492.0)
- removed the D21 at (677.5, 492.0)
- removed the D21 at (752.5, 492.0)
- removed the D22 at (820.0, 502.4)
- removed the D22 at (670.0, 502.4)
- removed the D22 at (595.0, 502.4)
- removed the D22 at (745.0, 502.4)
- removed the D23 at (581.9, 514.8)
- removed the D23 at (656.9, 514.8)
- removed the D23 at (806.9, 514.8)
- removed the D23 at (731.9, 514.8)
- removed the D3 at (566.4, 497.2)
- removed the D3 at (716.4, 497.2)
- removed the D3 at (641.4, 497.2)
- removed the D3 at (791.4, 497.2)
- removed the D4 at (566.3, 465.9)
- removed the D4 at (716.3, 465.9)
- removed the D4 at (641.3, 465.9)
- removed the D4 at (791.3, 465.9)
- removed the D5 at (811.4, 513.6)
- removed the D5 at (661.4, 513.6)
- removed the D5 at (586.4, 513.6)
- removed the D5 at (736.4, 513.6)
- removed the D6 at (644.0, 466.1)
- removed the D6 at (719.0, 466.1)
- removed the D6 at (794.0, 466.1)
- removed the D6 at (569.0, 466.1)
- removed the D7 at (856.1, 511.1)
- removed the D7 at (781.1, 511.1)
- removed the D7 at (706.1, 511.1)
- removed the D7 at (631.1, 511.1)
- removed the D8 at (722.0, 466.1)
- removed the D8 at (572.0, 466.1)
- removed the D8 at (647.0, 466.1)
- removed the D8 at (797.0, 466.1)
- removed the D9 at (643.7, 490.5)
- removed the D9 at (718.7, 490.5)
- removed the D9 at (568.7, 490.5)
- removed the D9 at (793.7, 490.5)
- removed the F1 at (656.5, 526.5)
- removed the F1 at (581.5, 526.5)
- removed the F1 at (806.5, 526.5)
- removed the F1 at (731.5, 526.5)
- removed the FID1 at (713.0, 450.5)
- removed the FID1 at (788.0, 450.5)
- removed the FID1 at (563.0, 450.5)
- removed the FID1 at (563.1, 314.7)
- removed the FID1 at (638.0, 450.5)
- removed the FID2 at (638.0, 536.5)
- removed the FID2 at (713.0, 536.5)
- removed the FID2 at (563.0, 536.5)
- removed the FID2 at (788.0, 536.5)
- removed the FID3 at (859.0, 450.5)
- removed the FID3 at (634.0, 450.5)
- removed the FID3 at (709.0, 450.5)
- removed the FID3 at (784.0, 450.5)
- removed the FID4 at (784.0, 450.5)
- removed the FID4 at (859.0, 450.5)
- removed the FID4 at (709.0, 450.5)
- removed the FID4 at (634.0, 450.5)
- removed the FID5 at (638.0, 536.5)
- removed the FID5 at (788.0, 536.5)
- removed the FID5 at (713.0, 536.5)
- removed the FID5 at (563.0, 536.5)
- removed the FID6 at (713.0, 450.5)
- removed the FID6 at (563.0, 450.5)
- removed the FID6 at (788.0, 450.5)
- removed the FID6 at (638.0, 450.5)
- removed the J1 at (826.4, 495.6)
- removed the J1 at (676.4, 495.6)
- removed the J1 at (751.4, 495.6)
- removed the J1 at (601.4, 495.6)
- removed the J10 at (706.9, 457.6)
- removed the J10 at (856.9, 457.6)
- removed the J10 at (631.9, 457.6)
- removed the J10 at (781.9, 457.6)
- removed the J11 at (820.4, 457.8)
- removed the J11 at (595.4, 457.8)
- removed the J11 at (745.4, 457.8)
- removed the J11 at (670.4, 457.8)
- removed the J2 at (779.6, 533.2)
- removed the J2 at (854.6, 533.2)
- removed the J2 at (629.6, 533.2)
- removed the J2 at (704.6, 533.2)
- removed the J3 at (700.4, 526.7)
- removed the J3 at (625.4, 526.7)
- removed the J3 at (775.4, 526.7)
- removed the J3 at (850.4, 526.7)
- removed the J4 at (769.1, 533.3)
- removed the J4 at (694.1, 533.3)
- removed the J4 at (619.1, 533.3)
- removed the J4 at (844.1, 533.3)
- removed the J5 at (685.0, 533.2)
- removed the J5 at (760.0, 533.2)
- removed the J5 at (610.0, 533.2)
- removed the J5 at (835.0, 533.2)
- removed the J6 at (781.8, 461.6)
- removed the J6 at (856.8, 461.6)
- removed the J6 at (631.8, 461.6)
- removed the J6 at (706.8, 461.6)
- removed the J7 at (855.9, 521.0)
- removed the J7 at (705.9, 521.0)
- removed the J7 at (780.9, 521.0)
- removed the J7 at (630.9, 521.0)
- removed the J9 at (583.0, 460.6)
- removed the J9 at (808.0, 460.6)
- removed the J9 at (658.0, 460.6)
- removed the J9 at (733.0, 460.6)
- removed the JP1 at (670.7, 497.0)
- removed the JP1 at (820.7, 497.0)
- removed the JP1 at (595.7, 497.0)
- removed the JP1 at (745.7, 497.0)
- removed the K2 at (645.8, 508.4)
- removed the K2 at (795.8, 508.4)
- removed the K2 at (720.8, 508.4)
- removed the K2 at (570.8, 508.4)
- removed the K3 at (572.1, 520.3)
- removed the K3 at (797.1, 520.3)
- removed the K3 at (647.1, 520.3)
- removed the K3 at (722.1, 520.3)
- removed the L1 at (700.1, 498.6)
- removed the L1 at (625.1, 498.6)
- removed the L1 at (775.1, 498.6)
- removed the L1 at (850.1, 498.6)
- removed the L2 at (812.5, 493.2)
- removed the L2 at (587.5, 493.2)
- removed the L2 at (662.5, 493.2)
- removed the L2 at (737.5, 493.2)
- removed the L5 at (836.5, 527.4)
- removed the L5 at (686.5, 527.4)
- removed the L5 at (611.5, 527.4)
- removed the L5 at (761.5, 527.4)
- removed the Q1 at (825.7, 502.6)
- removed the Q1 at (600.7, 502.6)
- removed the Q1 at (750.7, 502.6)
- removed the Q1 at (675.7, 502.6)
- removed the Q2 at (693.8, 481.6)
- removed the Q2 at (618.8, 481.6)
- removed the Q2 at (843.8, 481.6)
- removed the Q2 at (768.8, 481.6)
- removed the Q3 at (656.9, 515.6)
- removed the Q3 at (731.9, 515.6)
- removed the Q3 at (806.9, 515.6)
- removed the Q3 at (581.9, 515.6)
- removed the Q4 at (755.8, 500.2)
- removed the Q4 at (680.8, 500.2)
- removed the Q4 at (605.8, 500.2)
- removed the Q4 at (830.8, 500.2)
- removed the Q5 at (604.9, 478.5)
- removed the Q5 at (829.9, 478.5)
- removed the Q5 at (754.9, 478.5)
- removed the Q5 at (679.9, 478.5)
- removed the R10 at (769.1, 475.7)
- removed the R10 at (844.1, 475.7)
- removed the R10 at (619.1, 475.7)
- removed the R10 at (694.1, 475.7)
- removed the R11 at (769.2, 471.4)
- removed the R11 at (619.2, 471.4)
- removed the R11 at (694.2, 471.4)
- removed the R11 at (844.2, 471.4)
- removed the R12 at (622.4, 469.5)
- removed the R12 at (697.4, 469.5)
- removed the R12 at (847.4, 469.5)
- removed the R12 at (772.4, 469.5)
- removed the R13 at (624.1, 469.5)
- removed the R13 at (774.1, 469.5)
- removed the R13 at (699.1, 469.5)
- removed the R13 at (849.1, 469.5)
- removed the R14 at (642.0, 473.1)
- removed the R14 at (717.0, 473.1)
- removed the R14 at (792.0, 473.1)
- removed the R14 at (567.0, 473.1)
- removed the R15 at (764.6, 499.4)
- removed the R15 at (689.6, 499.4)
- removed the R15 at (614.6, 499.4)
- removed the R15 at (839.6, 499.4)
- removed the R16 at (844.1, 477.9)
- removed the R16 at (694.1, 477.9)
- removed the R16 at (769.1, 477.9)
- removed the R16 at (619.1, 477.9)
- removed the R17 at (759.3, 499.4)
- removed the R17 at (834.3, 499.4)
- removed the R17 at (609.3, 499.4)
- removed the R17 at (684.3, 499.4)
- removed the R18 at (705.0, 523.1)
- removed the R18 at (855.0, 523.1)
- removed the R18 at (780.0, 523.1)
- removed the R18 at (630.0, 523.1)
- removed the R19 at (702.4, 523.1)
- removed the R19 at (852.4, 523.1)
- removed the R19 at (777.4, 523.1)
- removed the R19 at (627.4, 523.1)
- removed the R20 at (670.1, 461.6)
- removed the R20 at (595.1, 461.6)
- removed the R20 at (745.1, 461.6)
- removed the R20 at (820.1, 461.6)
- removed the R21 at (855.8, 520.0)
- removed the R21 at (705.8, 520.0)
- removed the R21 at (780.8, 520.0)
- removed the R21 at (630.8, 520.0)
- removed the R22 at (769.5, 495.1)
- removed the R22 at (694.5, 495.1)
- removed the R22 at (619.5, 495.1)
- removed the R22 at (844.5, 495.1)
- removed the R23 at (701.0, 493.8)
- removed the R23 at (626.0, 493.8)
- removed the R23 at (776.0, 493.8)
- removed the R23 at (851.0, 493.8)
- removed the R24 at (670.2, 463.6)
- removed the R24 at (820.2, 463.6)
- removed the R24 at (745.2, 463.6)
- removed the R24 at (595.2, 463.6)
- removed the R25 at (770.3, 502.2)
- removed the R25 at (620.3, 502.2)
- removed the R25 at (695.3, 502.2)
- removed the R25 at (845.3, 502.2)
- removed the R26 at (691.4, 502.2)
- removed the R26 at (841.4, 502.2)
- removed the R26 at (616.4, 502.2)
- removed the R26 at (766.4, 502.2)
- removed the R27 at (853.4, 503.8)
- removed the R27 at (628.4, 503.8)
- removed the R27 at (703.4, 503.8)
- removed the R27 at (778.4, 503.8)
- removed the R28 at (752.5, 490.2)
- removed the R28 at (827.5, 490.2)
- removed the R28 at (602.5, 490.2)
- removed the R28 at (677.5, 490.2)
- removed the R29 at (752.4, 492.6)
- removed the R29 at (827.4, 492.6)
- removed the R29 at (602.4, 492.6)
- removed the R29 at (677.4, 492.6)
- removed the R3 at (811.6, 526.1)
- removed the R3 at (736.6, 526.1)
- removed the R3 at (661.6, 526.1)
- removed the R3 at (586.6, 526.1)
- removed the R30 at (684.9, 476.0)
- removed the R30 at (759.9, 476.0)
- removed the R30 at (834.9, 476.0)
- removed the R30 at (609.9, 476.0)
- removed the R31 at (773.7, 489.2)
- removed the R31 at (623.7, 489.2)
- removed the R31 at (698.7, 489.2)
- removed the R31 at (848.7, 489.2)
- removed the R32 at (703.8, 485.6)
- removed the R32 at (853.8, 485.6)
- removed the R32 at (778.8, 485.6)
- removed the R32 at (628.8, 485.6)
- removed the R33 at (754.8, 481.6)
- removed the R33 at (679.8, 481.6)
- removed the R33 at (604.8, 481.6)
- removed the R33 at (829.8, 481.6)
- removed the R34 at (852.5, 508.3)
- removed the R34 at (702.5, 508.3)
- removed the R34 at (627.5, 508.3)
- removed the R34 at (777.5, 508.3)
- removed the R35 at (777.6, 510.4)
- removed the R35 at (627.6, 510.4)
- removed the R35 at (852.6, 510.4)
- removed the R35 at (702.6, 510.4)
- removed the R36 at (735.3, 476.9)
- removed the R36 at (810.3, 476.9)
- removed the R36 at (660.3, 476.9)
- removed the R36 at (585.3, 476.9)
- removed the R37 at (731.9, 503.0)
- removed the R37 at (656.9, 503.0)
- removed the R37 at (806.9, 503.0)
- removed the R37 at (581.9, 503.0)
- removed the R38 at (585.5, 497.1)
- removed the R38 at (810.5, 497.1)
- removed the R38 at (660.5, 497.1)
- removed the R38 at (735.5, 497.1)
- removed the R39 at (656.7, 510.8)
- removed the R39 at (806.7, 510.8)
- removed the R39 at (731.7, 510.8)
- removed the R39 at (581.7, 510.8)
- removed the R4 at (589.5, 526.3)
- removed the R4 at (814.5, 526.3)
- removed the R4 at (664.5, 526.3)
- removed the R4 at (739.5, 526.3)
- removed the R40 at (810.6, 494.8)
- removed the R40 at (585.6, 494.8)
- removed the R40 at (735.6, 494.8)
- removed the R40 at (660.6, 494.8)
- removed the R41 at (720.2, 497.3)
- removed the R41 at (795.2, 497.3)
- removed the R41 at (645.2, 497.3)
- removed the R41 at (570.2, 497.3)
- removed the R42 at (645.2, 499.9)
- removed the R42 at (795.2, 499.9)
- removed the R42 at (570.2, 499.9)
- removed the R42 at (720.2, 499.9)
- removed the R43 at (829.3, 482.1)
- removed the R43 at (604.3, 482.1)
- removed the R43 at (754.3, 482.1)
- removed the R43 at (679.3, 482.1)
- removed the R44 at (758.4, 482.1)
- removed the R44 at (683.4, 482.1)
- removed the R44 at (608.4, 482.1)
- removed the R44 at (833.4, 482.1)
- removed the R45 at (778.5, 506.0)
- removed the R45 at (628.5, 506.0)
- removed the R45 at (853.5, 506.0)
- removed the R45 at (703.5, 506.0)
- removed the R47 at (748.3, 497.1)
- removed the R47 at (598.3, 497.1)
- removed the R47 at (823.3, 497.1)
- removed the R47 at (673.3, 497.1)
- removed the R49 at (598.3, 493.7)
- removed the R49 at (673.3, 493.7)
- removed the R49 at (823.3, 493.7)
- removed the R49 at (748.3, 493.7)
- removed the R5 at (567.0, 471.2)
- removed the R5 at (792.0, 471.2)
- removed the R5 at (642.0, 471.2)
- removed the R5 at (717.0, 471.2)
- removed the R50 at (744.6, 488.9)
- removed the R50 at (819.6, 488.9)
- removed the R50 at (669.6, 488.9)
- removed the R50 at (594.6, 488.9)
- removed the R51 at (664.0, 494.8)
- removed the R51 at (814.0, 494.8)
- removed the R51 at (589.0, 494.8)
- removed the R51 at (739.0, 494.8)
- removed the R52 at (672.2, 488.9)
- removed the R52 at (597.2, 488.9)
- removed the R52 at (822.2, 488.9)
- removed the R52 at (747.2, 488.9)
- removed the R53 at (592.3, 488.8)
- removed the R53 at (817.3, 488.8)
- removed the R53 at (742.3, 488.8)
- removed the R53 at (667.3, 488.8)
- removed the R54 at (837.6, 524.1)
- removed the R54 at (687.6, 524.1)
- removed the R54 at (762.6, 524.1)
- removed the R54 at (612.6, 524.1)
- removed the R6 at (567.0, 469.5)
- removed the R6 at (717.0, 469.5)
- removed the R6 at (792.0, 469.5)
- removed the R6 at (642.0, 469.5)
- removed the R7 at (642.1, 467.7)
- removed the R7 at (717.1, 467.7)
- removed the R7 at (567.1, 467.7)
- removed the R7 at (792.1, 467.7)
- removed the R8 at (631.2, 499.0)
- removed the R8 at (706.2, 499.0)
- removed the R8 at (856.2, 499.0)
- removed the R8 at (781.2, 499.0)
- removed the R9 at (706.2, 496.4)
- removed the R9 at (631.2, 496.4)
- removed the R9 at (781.2, 496.4)
- removed the R9 at (856.2, 496.4)
- removed the TP2 at (726.2, 461.8)
- removed the TP2 at (801.2, 461.8)
- removed the TP2 at (651.2, 461.8)
- removed the TP2 at (576.2, 461.8)
- removed the TP3 at (651.9, 470.6)
- removed the TP3 at (576.9, 470.6)
- removed the TP3 at (801.9, 470.6)
- removed the TP3 at (726.9, 470.6)
- removed the TP4 at (595.2, 501.1)
- removed the TP4 at (670.2, 501.1)
- removed the TP4 at (745.2, 501.1)
- removed the TP4 at (820.2, 501.1)
- removed the U11 at (819.1, 494.9)
- removed the U11 at (594.1, 494.9)
- removed the U11 at (669.1, 494.9)
- removed the U11 at (744.1, 494.9)
- removed the U12 at (728.1, 499.2)
- removed the U12 at (653.1, 499.2)
- removed the U12 at (803.1, 499.2)
- removed the U12 at (578.1, 499.2)
- removed the U13 at (595.0, 472.6)
- removed the U13 at (820.0, 472.6)
- removed the U13 at (745.0, 472.6)
- removed the U13 at (670.0, 472.6)
- removed the U14 at (841.1, 514.5)
- removed the U14 at (766.1, 514.5)
- removed the U14 at (616.1, 514.5)
- removed the U14 at (691.1, 514.5)
- removed the U2 at (719.5, 498.2)
- removed the U2 at (794.5, 498.2)
- removed the U2 at (644.5, 498.2)
- removed the U2 at (569.5, 498.2)
- removed the U3 at (758.6, 495.0)
- removed the U3 at (608.6, 495.0)
- removed the U3 at (833.6, 495.0)
- removed the U3 at (683.6, 495.0)
- removed the U4 at (568.5, 476.6)
- removed the U4 at (643.5, 476.6)
- removed the U4 at (793.5, 476.6)
- removed the U4 at (718.5, 476.6)
- removed the U5 at (839.8, 495.6)
- removed the U5 at (689.8, 495.6)
- removed the U5 at (764.8, 495.6)
- removed the U5 at (614.8, 495.6)
- removed the U6 at (621.0, 474.3)
- removed the U6 at (771.0, 474.3)
- removed the U6 at (696.0, 474.3)
- removed the U6 at (846.0, 474.3)
- removed the U7 at (691.1, 495.3)
- removed the U7 at (766.1, 495.3)
- removed the U7 at (841.1, 495.3)
- removed the U7 at (616.1, 495.3)
- removed the U8 at (841.2, 513.4)
- removed the U8 at (691.2, 513.4)
- removed the U8 at (616.2, 513.4)
- removed the U8 at (766.2, 513.4)
- removed the U9 at (736.9, 505.7)
- removed the U9 at (586.9, 505.7)
- removed the U9 at (661.9, 505.7)
- removed the U9 at (811.9, 505.7)
- removed the Y1 at (838.8, 485.2)
- removed the Y1 at (688.8, 485.2)
- removed the Y1 at (613.8, 485.2)
- removed the Y1 at (763.8, 485.2)
- removed the Y4 at (739.5, 484.8)
- removed the Y4 at (589.5, 484.8)
- removed the Y4 at (814.5, 484.8)
- removed the Y4 at (664.5, 484.8)
- removed the Y5 at (823.5, 486.1)
- removed the Y5 at (748.5, 486.1)
- removed the Y5 at (673.5, 486.1)
- removed the Y5 at (598.5, 486.1)
- added BT1: 1056, 1056:BAT_1056, B.Cu at (112.3, 124.5)
- added BT1: 1056, 1056:BAT_1056, B.Cu at (337.3, 124.5)
- added BT1: 1056, 1056:BAT_1056, B.Cu at (187.3, 124.5)
- added BT1: 1056, 1056:BAT_1056, B.Cu at (262.3, 124.5)
- added BZ1: Buzzer, Buzzer_Beeper:MagneticBuzzer_ProSignal_ABI-009-RC, F.Cu at (266.4, 122.8)
- added BZ1: Buzzer, Buzzer_Beeper:MagneticBuzzer_ProSignal_ABI-009-RC, F.Cu at (116.4, 122.8)
- added BZ1: Buzzer, Buzzer_Beeper:MagneticBuzzer_ProSignal_ABI-009-RC, F.Cu at (341.4, 122.8)
- added BZ1: Buzzer, Buzzer_Beeper:MagneticBuzzer_ProSignal_ABI-009-RC, F.Cu at (191.4, 122.8)
- added C1: 220uF/25V, Capacitor_SMD:CP_Elec_8x6.9, F.Cu at (238.7, 163.1)
- added C1: 220uF/25V, Capacitor_SMD:CP_Elec_8x6.9, F.Cu at (88.7, 163.1)
- added C1: 220uF/25V, Capacitor_SMD:CP_Elec_8x6.9, F.Cu at (163.7, 163.1)
- added C1: 220uF/25V, Capacitor_SMD:CP_Elec_8x6.9, F.Cu at (313.7, 163.1)
- added C10: 10uF/25V, Capacitor_THT:CP_Radial_D5.0mm_P2.50mm, F.Cu at (304.8, 136.0)
- added C10: 10uF/25V, Capacitor_THT:CP_Radial_D5.0mm_P2.50mm, F.Cu at (79.8, 136.0)
- added C10: 10uF/25V, Capacitor_THT:CP_Radial_D5.0mm_P2.50mm, F.Cu at (154.8, 136.0)
- added C10: 10uF/25V, Capacitor_THT:CP_Radial_D5.0mm_P2.50mm, F.Cu at (229.8, 136.0)
- added C11: 1uF/16V, Capacitor_SMD:C_0603_1608Metric, B.Cu at (230.5, 139.2)
- added C11: 1uF/16V, Capacitor_SMD:C_0603_1608Metric, B.Cu at (80.5, 139.2)
- added C11: 1uF/16V, Capacitor_SMD:C_0603_1608Metric, B.Cu at (155.5, 139.2)
- added C11: 1uF/16V, Capacitor_SMD:C_0603_1608Metric, B.Cu at (305.5, 139.2)
- added C12: 0.1uF/16V, Capacitor_SMD:C_0603_1608Metric, F.Cu at (282.6, 151.8)
- added C12: 0.1uF/16V, Capacitor_SMD:C_0603_1608Metric, F.Cu at (207.6, 151.8)
- added C12: 0.1uF/16V, Capacitor_SMD:C_0603_1608Metric, F.Cu at (357.6, 151.8)
- added C12: 0.1uF/16V, Capacitor_SMD:C_0603_1608Metric, F.Cu at (132.6, 151.8)
- added C13: 100uFx6.3v, Capacitor_SMD:C_Elec_5x5.8, F.Cu at (177.3, 182.8)
- added C13: 100uFx6.3v, Capacitor_SMD:C_Elec_5x5.8, F.Cu at (252.3, 182.8)
- added C13: 100uFx6.3v, Capacitor_SMD:C_Elec_5x5.8, F.Cu at (327.3, 182.8)
- added C13: 100uFx6.3v, Capacitor_SMD:C_Elec_5x5.8, F.Cu at (102.3, 182.8)
- added C14: 220uF/10v, Capacitor_SMD:CP_Elec_8x6.5, F.Cu at (172.4, 174.2)
- added C14: 220uF/10v, Capacitor_SMD:CP_Elec_8x6.5, F.Cu at (322.4, 174.2)
- added C14: 220uF/10v, Capacitor_SMD:CP_Elec_8x6.5, F.Cu at (97.4, 174.2)
- added C14: 220uF/10v, Capacitor_SMD:CP_Elec_8x6.5, F.Cu at (247.4, 174.2)
- added C15: 0.1uFx/10V, Capacitor_SMD:C_0805_2012Metric, F.Cu at (173.0, 165.4)
- added C15: 0.1uFx/10V, Capacitor_SMD:C_0805_2012Metric, F.Cu at (98.0, 165.4)
- added C15: 0.1uFx/10V, Capacitor_SMD:C_0805_2012Metric, F.Cu at (248.0, 165.4)
- added C15: 0.1uFx/10V, Capacitor_SMD:C_0805_2012Metric, F.Cu at (323.0, 165.4)
- added C16: 1uF, Capacitor_SMD:C_0603_1608Metric, F.Cu at (186.9, 144.2)
- added C16: 1uF, Capacitor_SMD:C_0603_1608Metric, F.Cu at (336.9, 144.2)
- added C16: 1uF, Capacitor_SMD:C_0603_1608Metric, F.Cu at (111.9, 144.2)
- added C16: 1uF, Capacitor_SMD:C_0603_1608Metric, F.Cu at (261.9, 144.2)
- added C17: 18pF, Capacitor_SMD:C_0603_1608Metric, F.Cu at (339.6, 139.6)
- added C17: 18pF, Capacitor_SMD:C_0603_1608Metric, F.Cu at (264.6, 139.6)
- added C17: 18pF, Capacitor_SMD:C_0603_1608Metric, F.Cu at (114.6, 139.6)
- added C17: 18pF, Capacitor_SMD:C_0603_1608Metric, F.Cu at (189.6, 139.6)
- added C18: 18pF, Capacitor_SMD:C_0603_1608Metric, F.Cu at (267.7, 139.6)
- added C18: 18pF, Capacitor_SMD:C_0603_1608Metric, F.Cu at (192.7, 139.6)
- added C18: 18pF, Capacitor_SMD:C_0603_1608Metric, F.Cu at (342.7, 139.6)
- added C18: 18pF, Capacitor_SMD:C_0603_1608Metric, F.Cu at (117.7, 139.6)
- added C19: 1uF/6.3V, Capacitor_SMD:C_0603_1608Metric, F.Cu at (178.9, 119.9)
- added C19: 1uF/6.3V, Capacitor_SMD:C_0603_1608Metric, F.Cu at (253.9, 119.9)
- added C19: 1uF/6.3V, Capacitor_SMD:C_0603_1608Metric, F.Cu at (328.9, 119.9)
- added C19: 1uF/6.3V, Capacitor_SMD:C_0603_1608Metric, F.Cu at (103.9, 119.9)
- added C2: 10uFx16v, Capacitor_SMD:C_0603_1608Metric, B.Cu at (355.5, 164.3)
- added C2: 10uFx16v, Capacitor_SMD:C_0603_1608Metric, B.Cu at (280.5, 164.3)
- added C2: 10uFx16v, Capacitor_SMD:C_0603_1608Metric, B.Cu at (205.5, 164.3)
- added C2: 10uFx16v, Capacitor_SMD:C_0603_1608Metric, B.Cu at (130.5, 164.3)
- added C20: 0.1uF/6.3V, Capacitor_SMD:C_0603_1608Metric, F.Cu at (178.9, 121.7)
- added C20: 0.1uF/6.3V, Capacitor_SMD:C_0603_1608Metric, F.Cu at (328.9, 121.7)
- added C20: 0.1uF/6.3V, Capacitor_SMD:C_0603_1608Metric, F.Cu at (103.9, 121.7)
- added C20: 0.1uF/6.3V, Capacitor_SMD:C_0603_1608Metric, F.Cu at (253.9, 121.7)
- added C21: 1uF/6.3V, Capacitor_SMD:C_0603_1608Metric, F.Cu at (319.9, 121.6)
- added C21: 1uF/6.3V, Capacitor_SMD:C_0603_1608Metric, F.Cu at (94.9, 121.6)
- added C21: 1uF/6.3V, Capacitor_SMD:C_0603_1608Metric, F.Cu at (169.9, 121.6)
- added C21: 1uF/6.3V, Capacitor_SMD:C_0603_1608Metric, F.Cu at (244.9, 121.6)
- added C22: 0.1uF/6.3V, Capacitor_SMD:C_0603_1608Metric, F.Cu at (244.8, 119.7)
- added C22: 0.1uF/6.3V, Capacitor_SMD:C_0603_1608Metric, F.Cu at (319.8, 119.7)
- added C22: 0.1uF/6.3V, Capacitor_SMD:C_0603_1608Metric, F.Cu at (94.8, 119.7)
- added C22: 0.1uF/6.3V, Capacitor_SMD:C_0603_1608Metric, F.Cu at (169.8, 119.7)
- added C23: 1uF/6.3V, Capacitor_SMD:C_0603_1608Metric, F.Cu at (164.1, 140.5)
- added C23: 1uF/6.3V, Capacitor_SMD:C_0603_1608Metric, F.Cu at (314.1, 140.5)
- added C23: 1uF/6.3V, Capacitor_SMD:C_0603_1608Metric, F.Cu at (89.1, 140.5)
- added C23: 1uF/6.3V, Capacitor_SMD:C_0603_1608Metric, F.Cu at (239.1, 140.5)
- added C24: 0.1uF/6.3V, Capacitor_SMD:C_0603_1608Metric, F.Cu at (313.3, 136.6)
- added C24: 0.1uF/6.3V, Capacitor_SMD:C_0603_1608Metric, F.Cu at (88.3, 136.6)
- added C24: 0.1uF/6.3V, Capacitor_SMD:C_0603_1608Metric, F.Cu at (163.3, 136.6)
- added C24: 0.1uF/6.3V, Capacitor_SMD:C_0603_1608Metric, F.Cu at (238.3, 136.6)
- added C25: 1uF/6.3V, Capacitor_SMD:C_0603_1608Metric, F.Cu at (257.7, 135.6)
- added C25: 1uF/6.3V, Capacitor_SMD:C_0603_1608Metric, F.Cu at (107.7, 135.6)
- added C25: 1uF/6.3V, Capacitor_SMD:C_0603_1608Metric, F.Cu at (182.7, 135.6)
- added C25: 1uF/6.3V, Capacitor_SMD:C_0603_1608Metric, F.Cu at (332.7, 135.6)
- added C26: 0.1uF/6.3V, Capacitor_SMD:C_0603_1608Metric, F.Cu at (259.6, 135.7)
- added C26: 0.1uF/6.3V, Capacitor_SMD:C_0603_1608Metric, F.Cu at (184.6, 135.7)
- added C26: 0.1uF/6.3V, Capacitor_SMD:C_0603_1608Metric, F.Cu at (334.6, 135.7)
- added C26: 0.1uF/6.3V, Capacitor_SMD:C_0603_1608Metric, F.Cu at (109.6, 135.7)
- added C27: 0.1uFx/10V, Capacitor_SMD:C_0805_2012Metric, F.Cu at (253.5, 168.0)
- added C27: 0.1uFx/10V, Capacitor_SMD:C_0805_2012Metric, F.Cu at (178.5, 168.0)
- added C27: 0.1uFx/10V, Capacitor_SMD:C_0805_2012Metric, F.Cu at (328.5, 168.0)
- added C27: 0.1uFx/10V, Capacitor_SMD:C_0805_2012Metric, F.Cu at (103.5, 168.0)
- added C28: 1uF/6.3V, Capacitor_SMD:C_0603_1608Metric, F.Cu at (262.1, 131.6)
- added C28: 1uF/6.3V, Capacitor_SMD:C_0603_1608Metric, F.Cu at (112.0, 131.6)
- added C28: 1uF/6.3V, Capacitor_SMD:C_0603_1608Metric, F.Cu at (187.1, 131.6)
- added C28: 1uF/6.3V, Capacitor_SMD:C_0603_1608Metric, F.Cu at (337.1, 131.6)
- added C29: 0.1uF/6.3V, Capacitor_SMD:C_0603_1608Metric, F.Cu at (188.7, 131.6)
- added C29: 0.1uF/6.3V, Capacitor_SMD:C_0603_1608Metric, F.Cu at (113.7, 131.6)
- added C29: 0.1uF/6.3V, Capacitor_SMD:C_0603_1608Metric, F.Cu at (338.7, 131.6)
- added C29: 0.1uF/6.3V, Capacitor_SMD:C_0603_1608Metric, F.Cu at (263.7, 131.6)
- added C30: 1uF/6.3V, Capacitor_SMD:C_0603_1608Metric, F.Cu at (207.8, 129.3)
- added C30: 1uF/6.3V, Capacitor_SMD:C_0603_1608Metric, F.Cu at (282.8, 129.3)
- added C30: 1uF/6.3V, Capacitor_SMD:C_0603_1608Metric, F.Cu at (132.8, 129.3)
- added C30: 1uF/6.3V, Capacitor_SMD:C_0603_1608Metric, F.Cu at (357.8, 129.3)
- added C31: 0.1uF/6.3V, Capacitor_SMD:C_0603_1608Metric, F.Cu at (134.9, 129.3)
- added C31: 0.1uF/6.3V, Capacitor_SMD:C_0603_1608Metric, F.Cu at (209.9, 129.3)
- added C31: 0.1uF/6.3V, Capacitor_SMD:C_0603_1608Metric, F.Cu at (284.9, 129.3)
- added C31: 0.1uF/6.3V, Capacitor_SMD:C_0603_1608Metric, F.Cu at (359.9, 129.3)
- added C32: 0.1uF, Capacitor_SMD:C_0603_1608Metric, B.Cu at (238.5, 157.1)
- added C32: 0.1uF, Capacitor_SMD:C_0603_1608Metric, B.Cu at (88.5, 157.1)
- added C32: 0.1uF, Capacitor_SMD:C_0603_1608Metric, B.Cu at (313.5, 157.1)
- added C32: 0.1uF, Capacitor_SMD:C_0603_1608Metric, B.Cu at (163.5, 157.1)
- added C33: 0.1uF, Capacitor_SMD:C_0603_1608Metric, B.Cu at (173.3, 165.8)
- added C33: 0.1uF, Capacitor_SMD:C_0603_1608Metric, B.Cu at (98.3, 165.8)
- added C33: 0.1uF, Capacitor_SMD:C_0603_1608Metric, B.Cu at (248.3, 165.8)
- added C33: 0.1uF, Capacitor_SMD:C_0603_1608Metric, B.Cu at (323.3, 165.8)
- added C34: 0.1uF, Capacitor_SMD:C_0603_1608Metric, B.Cu at (320.6, 166.7)
- added C34: 0.1uF, Capacitor_SMD:C_0603_1608Metric, B.Cu at (95.5, 166.7)
- added C34: 0.1uF, Capacitor_SMD:C_0603_1608Metric, B.Cu at (245.6, 166.7)
- added C34: 0.1uF, Capacitor_SMD:C_0603_1608Metric, B.Cu at (170.6, 166.7)
- added C35: 0.1uF, Capacitor_SMD:C_0603_1608Metric, B.Cu at (92.0, 157.1)
- added C35: 0.1uF, Capacitor_SMD:C_0603_1608Metric, B.Cu at (317.0, 157.1)
- added C35: 0.1uF, Capacitor_SMD:C_0603_1608Metric, B.Cu at (167.0, 157.1)
- added C35: 0.1uF, Capacitor_SMD:C_0603_1608Metric, B.Cu at (242.0, 157.1)
- added C36: 0.1uF, Capacitor_SMD:C_0603_1608Metric, B.Cu at (242.0, 155.2)
- added C36: 0.1uF, Capacitor_SMD:C_0603_1608Metric, B.Cu at (317.0, 155.2)
- added C36: 0.1uF, Capacitor_SMD:C_0603_1608Metric, B.Cu at (92.0, 155.2)
- added C36: 0.1uF, Capacitor_SMD:C_0603_1608Metric, B.Cu at (167.0, 155.2)
- added C37: 22pF, Capacitor_SMD:C_0603_1608Metric, F.Cu at (321.4, 143.0)
- added C37: 22pF, Capacitor_SMD:C_0603_1608Metric, F.Cu at (171.3, 143.0)
- added C37: 22pF, Capacitor_SMD:C_0603_1608Metric, F.Cu at (96.3, 143.0)
- added C37: 22pF, Capacitor_SMD:C_0603_1608Metric, F.Cu at (246.3, 143.0)
- added C38: 330uF, Capacitor_Tantalum_SMD:CP_EIA-6032-15_Kemet-U, F.Cu at (104.4, 175.1)
- added C38: 330uF, Capacitor_Tantalum_SMD:CP_EIA-6032-15_Kemet-U, F.Cu at (179.4, 175.1)
- added C38: 330uF, Capacitor_Tantalum_SMD:CP_EIA-6032-15_Kemet-U, F.Cu at (329.4, 175.1)
- added C38: 330uF, Capacitor_Tantalum_SMD:CP_EIA-6032-15_Kemet-U, F.Cu at (254.4, 175.1)
- added C39: 10uFx/10V, Capacitor_SMD:C_0603_1608Metric, F.Cu at (178.6, 165.1)
- added C39: 10uFx/10V, Capacitor_SMD:C_0603_1608Metric, F.Cu at (103.6, 165.1)
- added C39: 10uFx/10V, Capacitor_SMD:C_0603_1608Metric, F.Cu at (253.6, 165.1)
- added C39: 10uFx/10V, Capacitor_SMD:C_0603_1608Metric, F.Cu at (328.6, 165.1)
- added C4: 220uF/25V, Capacitor_SMD:CP_Elec_8x6.9, F.Cu at (72.9, 143.6)
- added C4: 220uF/25V, Capacitor_SMD:CP_Elec_8x6.9, F.Cu at (147.9, 143.6)
- added C4: 220uF/25V, Capacitor_SMD:CP_Elec_8x6.9, F.Cu at (297.9, 143.6)
- added C4: 220uF/25V, Capacitor_SMD:CP_Elec_8x6.9, F.Cu at (222.9, 143.6)
- added C40: 22pF, Capacitor_SMD:C_0603_1608Metric, F.Cu at (171.4, 141.5)
- added C40: 22pF, Capacitor_SMD:C_0603_1608Metric, F.Cu at (321.4, 141.5)
- added C40: 22pF, Capacitor_SMD:C_0603_1608Metric, F.Cu at (96.4, 141.5)
- added C40: 22pF, Capacitor_SMD:C_0603_1608Metric, F.Cu at (246.4, 141.5)
- added C41: 18pF, Capacitor_SMD:C_0603_1608Metric, F.Cu at (326.3, 140.4)
- added C41: 18pF, Capacitor_SMD:C_0603_1608Metric, F.Cu at (251.3, 140.4)
- added C41: 18pF, Capacitor_SMD:C_0603_1608Metric, F.Cu at (101.3, 140.4)
- added C41: 18pF, Capacitor_SMD:C_0603_1608Metric, F.Cu at (176.3, 140.4)
- added C42: 18pF, Capacitor_SMD:C_0603_1608Metric, F.Cu at (179.3, 140.5)
- added C42: 18pF, Capacitor_SMD:C_0603_1608Metric, F.Cu at (329.3, 140.5)
- added C42: 18pF, Capacitor_SMD:C_0603_1608Metric, F.Cu at (104.3, 140.5)
- added C42: 18pF, Capacitor_SMD:C_0603_1608Metric, F.Cu at (254.3, 140.5)
- added C43: 1uF/6.3V, Capacitor_SMD:C_0603_1608Metric, F.Cu at (354.1, 147.2)
- added C43: 1uF/6.3V, Capacitor_SMD:C_0603_1608Metric, F.Cu at (204.2, 147.2)
- added C43: 1uF/6.3V, Capacitor_SMD:C_0603_1608Metric, F.Cu at (279.1, 147.2)
- added C43: 1uF/6.3V, Capacitor_SMD:C_0603_1608Metric, F.Cu at (129.2, 147.2)
- added C44: 0.1uF/6.3V, Capacitor_SMD:C_0603_1608Metric, F.Cu at (206.8, 147.2)
- added C44: 0.1uF/6.3V, Capacitor_SMD:C_0603_1608Metric, F.Cu at (131.8, 147.2)
- added C44: 0.1uF/6.3V, Capacitor_SMD:C_0603_1608Metric, F.Cu at (281.8, 147.2)
- added C44: 0.1uF/6.3V, Capacitor_SMD:C_0603_1608Metric, F.Cu at (356.8, 147.2)
- added C45: 1uF/6.3V, Capacitor_SMD:C_0603_1608Metric, F.Cu at (337.9, 135.8)
- added C45: 1uF/6.3V, Capacitor_SMD:C_0603_1608Metric, F.Cu at (113.0, 135.8)
- added C45: 1uF/6.3V, Capacitor_SMD:C_0603_1608Metric, F.Cu at (187.9, 135.8)
- added C45: 1uF/6.3V, Capacitor_SMD:C_0603_1608Metric, F.Cu at (262.9, 135.8)
- added C46: 0.1uF/6.3V, Capacitor_SMD:C_0603_1608Metric, F.Cu at (337.9, 137.7)
- added C46: 0.1uF/6.3V, Capacitor_SMD:C_0603_1608Metric, F.Cu at (187.9, 137.7)
- added C46: 0.1uF/6.3V, Capacitor_SMD:C_0603_1608Metric, F.Cu at (112.9, 137.7)
- added C46: 0.1uF/6.3V, Capacitor_SMD:C_0603_1608Metric, F.Cu at (262.9, 137.7)
- added C47: 1uF, Capacitor_SMD:C_0603_1608Metric, B.Cu at (323.1, 162.3)
- added C47: 1uF, Capacitor_SMD:C_0603_1608Metric, B.Cu at (173.1, 162.3)
- added C47: 1uF, Capacitor_SMD:C_0603_1608Metric, B.Cu at (98.1, 162.3)
- added C47: 1uF, Capacitor_SMD:C_0603_1608Metric, B.Cu at (248.1, 162.3)
- added C5: 1uF, Capacitor_SMD:C_0603_1608Metric, B.Cu at (87.3, 139.3)
- added C5: 1uF, Capacitor_SMD:C_0603_1608Metric, B.Cu at (237.3, 139.3)
- added C5: 1uF, Capacitor_SMD:C_0603_1608Metric, B.Cu at (162.3, 139.3)
- added C5: 1uF, Capacitor_SMD:C_0603_1608Metric, B.Cu at (312.3, 139.3)
- added C6: 1uF, Capacitor_SMD:C_0603_1608Metric, F.Cu at (157.0, 149.0)
- added C6: 1uF, Capacitor_SMD:C_0603_1608Metric, F.Cu at (82.0, 149.0)
- added C6: 1uF, Capacitor_SMD:C_0603_1608Metric, F.Cu at (232.0, 149.0)
- added C6: 1uF, Capacitor_SMD:C_0603_1608Metric, F.Cu at (307.0, 149.0)
- added C7: 10uF/16V, Capacitor_SMD:C_0603_1608Metric, F.Cu at (134.3, 159.4)
- added C7: 10uF/16V, Capacitor_SMD:C_0603_1608Metric, F.Cu at (284.3, 159.4)
- added C7: 10uF/16V, Capacitor_SMD:C_0603_1608Metric, F.Cu at (359.3, 159.4)
- added C7: 10uF/16V, Capacitor_SMD:C_0603_1608Metric, F.Cu at (209.3, 159.4)
- added C8: 10uF/16V, Capacitor_SMD:C_0603_1608Metric, F.Cu at (135.0, 163.0)
- added C8: 10uF/16V, Capacitor_SMD:C_0603_1608Metric, F.Cu at (285.0, 163.0)
- added C8: 10uF/16V, Capacitor_SMD:C_0603_1608Metric, F.Cu at (360.0, 163.0)
- added C8: 10uF/16V, Capacitor_SMD:C_0603_1608Metric, F.Cu at (210.0, 163.0)
- added C9: 10uF/25V, Capacitor_THT:CP_Radial_D5.0mm_P2.50mm, F.Cu at (231.7, 142.0)
- added C9: 10uF/25V, Capacitor_THT:CP_Radial_D5.0mm_P2.50mm, F.Cu at (306.7, 142.0)
- added C9: 10uF/25V, Capacitor_THT:CP_Radial_D5.0mm_P2.50mm, F.Cu at (156.7, 142.0)
- added C9: 10uF/25V, Capacitor_THT:CP_Radial_D5.0mm_P2.50mm, F.Cu at (81.7, 142.0)
- added CN1: Main_Connector, 66201821122:66201821122, F.Cu at (242.9, 190.6)
- added CN1: Main_Connector, 66201821122:66201821122, F.Cu at (92.9, 190.6)
- added CN1: Main_Connector, 66201821122:66201821122, F.Cu at (317.9, 190.6)
- added CN1: Main_Connector, 66201821122:66201821122, F.Cu at (167.9, 190.6)
- added D1: 3.9 Zener, Diode_SMD:D_SOD-123, F.Cu at (314.7, 178.4)
- added D1: 3.9 Zener, Diode_SMD:D_SOD-123, F.Cu at (164.7, 178.4)
- added D1: 3.9 Zener, Diode_SMD:D_SOD-123, F.Cu at (239.7, 178.4)
- added D1: 3.9 Zener, Diode_SMD:D_SOD-123, F.Cu at (89.7, 178.4)
- added D10: 3.9 Zener, Diode_SMD:D_SOD-123, B.Cu at (348.0, 131.5)
- added D10: 3.9 Zener, Diode_SMD:D_SOD-123, B.Cu at (198.0, 131.5)
- added D10: 3.9 Zener, Diode_SMD:D_SOD-123, B.Cu at (273.0, 131.5)
- added D10: 3.9 Zener, Diode_SMD:D_SOD-123, B.Cu at (123.0, 131.5)
- added D11: 3.9 Zener, Diode_SMD:D_SOD-123, B.Cu at (204.1, 128.3)
- added D11: 3.9 Zener, Diode_SMD:D_SOD-123, B.Cu at (279.1, 128.3)
- added D11: 3.9 Zener, Diode_SMD:D_SOD-123, B.Cu at (129.1, 128.3)
- added D11: 3.9 Zener, Diode_SMD:D_SOD-123, B.Cu at (354.1, 128.3)
- added D12: PW_LED, LED_SMD:LED_0805_2012Metric, F.Cu at (70.1, 128.3)
- added D12: PW_LED, LED_SMD:LED_0805_2012Metric, F.Cu at (295.1, 128.3)
- added D12: PW_LED, LED_SMD:LED_0805_2012Metric, F.Cu at (220.1, 128.3)
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Routing:
- removed copper zone on B.Cu, net (none)
- removed copper zone on F.Cu, net (none)
Other:
- board size 320 x 255 mm -> 320 x 136 mm
