File: Gov_TrkU_panel/Gov_tracker_Panel/Gov_tracker_Panel.kicad_pcb (KiCad board)
At the start: 2 copper layers, 320 x 136 mm, 689 parts, among them CN1 Main_Connector, J1 Conn_01x02, J10 Prog_T, J11 Debug, J2 USB_B_Mini, J3 USB_Con, J4 ANT, J5 Conn_Coaxial, J6 Debug/GPS_DBG, J7 Conn_Coaxial, J9 Prog_G, K2 G5Q-1, K3 SRA-05VDC-CL, Q1 SI2333DS, Q2 BC817, Q3 BC817, Q4 BSS84, Q5 BC817, U11 LM393, U12 W25Q128JVS, U13 STM32F103RCTx, U14 NEO-6M-GPS, U2 LM2596S-5, U3 SY7208B, U4 LM1117-3.3, U5 MCP73831-5-OT, U6 STM32F103RCTx, U7 693021020811, U8 SIM800C, U9 MAX3232, Y1 8MHz, Y4 32.678kHz, Y5 8MHz

Commit message: updated the diode positioning
Parts:
- removed the 3.3V at (154.9, 128.7)
- removed the 3.3V at (304.9, 128.7)
- removed the 3.3V at (229.9, 128.7)
- removed the 5V at (154.2, 119.8)
- removed the 5V at (229.2, 119.8)
- removed the 5V at (304.2, 119.8)
- removed the BT1 at (187.3, 124.5)
- removed the BT1 at (337.3, 124.5)
- removed the BT1 at (262.3, 124.5)
- removed the BZ1 at (191.4, 122.8)
- removed the BZ1 at (266.4, 122.8)
- removed the BZ1 at (341.4, 122.8)
- removed the C1 at (163.7, 163.1)
- removed the C1 at (238.7, 163.1)
- removed the C1 at (313.7, 163.1)
- removed the C10 at (154.8, 136.0)
- removed the C10 at (229.8, 136.0)
- removed the C10 at (304.8, 136.0)
- removed the C11 at (155.5, 139.2)
- removed the C11 at (230.5, 139.2)
- removed the C11 at (305.5, 139.2)
- removed the C12 at (282.6, 151.8)
- removed the C12 at (207.6, 151.8)
- removed the C12 at (357.6, 151.8)
- removed the C13 at (174.0, 183.0)
- removed the C13 at (249.0, 183.0)
- removed the C13 at (324.0, 183.0)
- removed the C14 at (172.4, 174.2)
- removed the C14 at (247.4, 174.2)
- removed the C14 at (322.4, 174.2)
- removed the C15 at (173.0, 165.4)
- removed the C15 at (323.0, 165.4)
- removed the C15 at (248.0, 165.4)
- removed the C16 at (336.9, 144.2)
- removed the C16 at (261.9, 144.2)
- removed the C16 at (186.9, 144.2)
- removed the C17 at (193.0, 141.5)
- removed the C17 at (268.0, 141.5)
- removed the C17 at (343.0, 141.5)
- removed the C18 at (271.8, 141.6)
- removed the C18 at (196.8, 141.6)
- removed the C18 at (346.8, 141.6)
- removed the C19 at (178.9, 119.9)
- removed the C19 at (253.9, 119.9)
- removed the C19 at (328.9, 119.9)
- removed the C2 at (280.5, 164.3)
- removed the C2 at (355.5, 164.3)
- removed the C2 at (205.5, 164.3)
- removed the C20 at (178.9, 121.7)
- removed the C20 at (328.9, 121.7)
- removed the C20 at (253.9, 121.7)
- removed the C21 at (244.9, 121.6)
- removed the C21 at (169.9, 121.6)
- removed the C21 at (319.9, 121.6)
- removed the C22 at (319.8, 119.7)
- removed the C22 at (169.8, 119.7)
- removed the C22 at (244.8, 119.7)
- removed the C23 at (239.1, 140.5)
- removed the C23 at (164.1, 140.5)
- removed the C23 at (314.1, 140.5)
- removed the C24 at (163.3, 136.6)
- removed the C24 at (238.3, 136.6)
- removed the C24 at (313.3, 136.6)
- removed the C25 at (182.7, 135.6)
- removed the C25 at (257.7, 135.6)
- removed the C25 at (332.7, 135.6)
- removed the C26 at (259.6, 135.7)
- removed the C26 at (334.6, 135.7)
- removed the C26 at (184.6, 135.7)
- removed the C27 at (178.5, 168.0)
- removed the C27 at (253.5, 168.0)
- removed the C27 at (328.5, 168.0)
- removed the C28 at (262.1, 131.6)
- removed the C28 at (187.1, 131.6)
- removed the C28 at (337.1, 131.6)
- removed the C29 at (263.7, 131.6)
- removed the C29 at (338.7, 131.6)
- removed the C29 at (188.7, 131.6)
- removed the C30 at (207.8, 129.3)
- removed the C30 at (282.8, 129.3)
- removed the C30 at (357.8, 129.3)
- removed the C31 at (209.9, 129.3)
- removed the C31 at (284.9, 129.3)
- removed the C31 at (359.9, 129.3)
- removed the C32 at (163.5, 157.1)
- removed the C32 at (238.5, 157.1)
- removed the C32 at (313.5, 157.1)
- removed the C33 at (323.3, 165.8)
- removed the C33 at (173.3, 165.8)
- removed the C33 at (248.3, 165.8)
- removed the C34 at (320.6, 166.7)
- removed the C34 at (170.6, 166.7)
- removed the C34 at (245.6, 166.7)
- removed the C35 at (317.0, 157.1)
- removed the C35 at (242.0, 157.1)
- removed the C35 at (167.0, 157.1)
- removed the C36 at (167.0, 155.2)
- removed the C36 at (317.0, 155.2)
- removed the C36 at (242.0, 155.2)
- removed the C37 at (320.3, 140.3)
- removed the C37 at (245.3, 140.3)
- removed the C37 at (170.3, 140.3)
- removed the C38 at (254.0, 173.2)
- removed the C38 at (179.0, 173.2)
- removed the C38 at (329.0, 173.2)
- removed the C39 at (178.6, 165.1)
- removed the C39 at (253.6, 165.1)
- removed the C39 at (328.6, 165.1)
- removed the C4 at (147.9, 143.6)
- removed the C4 at (222.9, 143.6)
- removed the C4 at (297.9, 143.6)
- removed the C40 at (242.2, 140.3)
- removed the C40 at (317.2, 140.3)
- removed the C40 at (167.2, 140.3)
- removed the C41 at (323.4, 140.3)
- removed the C41 at (173.4, 140.3)
- removed the C41 at (248.4, 140.3)
- removed the C42 at (251.5, 140.3)
- removed the C42 at (176.5, 140.3)
- removed the C42 at (326.5, 140.3)
- removed the C43 at (279.1, 147.2)
- removed the C43 at (354.1, 147.2)
- removed the C43 at (204.2, 147.2)
- removed the C44 at (356.8, 147.2)
- removed the C44 at (206.8, 147.2)
- removed the C44 at (281.8, 147.2)
- removed the C45 at (337.9, 135.8)
- removed the C45 at (262.9, 135.8)
- removed the C45 at (187.9, 135.8)
- removed the C46 at (187.9, 137.7)
- removed the C46 at (262.9, 137.7)
- removed the C46 at (337.9, 137.7)
- removed the C47 at (173.1, 162.3)
- removed the C47 at (323.1, 162.3)
- removed the C47 at (248.1, 162.3)
- removed the C5 at (312.3, 139.3)
- removed the C5 at (237.3, 139.3)
- removed the C5 at (162.3, 139.3)
- removed the C6 at (307.0, 149.0)
- removed the C6 at (232.0, 149.0)
- removed the C6 at (157.0, 149.0)
- removed the C7 at (209.3, 159.4)
- removed the C7 at (359.3, 159.4)
- removed the C7 at (284.3, 159.4)
- removed the C8 at (285.0, 163.0)
- removed the C8 at (360.0, 163.0)
- removed the C8 at (210.0, 163.0)
- removed the C9 at (231.7, 142.0)
- removed the C9 at (156.7, 142.0)
- removed the C9 at (306.7, 142.0)
- removed the CN1 at (317.9, 190.6)
- removed the CN1 at (242.9, 190.6)
- removed the CN1 at (167.9, 190.6)
- removed the D1 at (164.7, 178.4)
- removed the D1 at (314.7, 178.4)
- removed the D1 at (239.7, 178.4)
- removed the D10 at (198.0, 131.5)
- removed the D10 at (348.0, 131.5)
- removed the D10 at (273.0, 131.5)
- removed the D11 at (204.1, 128.3)
- removed the D11 at (354.1, 128.3)
- removed the D11 at (279.1, 128.3)
- removed the D12 at (295.1, 128.3)
- removed the D12 at (220.1, 128.3)
- removed the D12 at (145.1, 128.3)
- removed the D13 at (346.9, 156.2)
- removed the D13 at (271.9, 156.2)
- removed the D13 at (196.9, 156.2)
- removed the D14 at (361.9, 180.0)
- removed the D14 at (136.9, 180.0)
- removed the D14 at (286.9, 180.0)
- removed the D14 at (211.9, 180.0)
- removed the D15 at (315.8, 121.2)
- removed the D15 at (165.8, 121.2)
- removed the D15 at (240.8, 121.2)
- removed the D16 at (328.4, 162.7)
- removed the D16 at (253.4, 162.7)
- removed the D16 at (178.4, 162.7)
- removed the D17 at (358.8, 173.3)
- removed the D17 at (208.8, 173.3)
- removed the D17 at (283.8, 173.3)
- removed the D18 at (208.7, 170.3)
- removed the D18 at (283.7, 170.3)
- removed the D18 at (358.7, 170.3)
- removed the D19 at (236.9, 139.9)
- removed the D19 at (311.9, 139.9)
- removed the D19 at (161.9, 139.9)
- removed the D2 at (300.3, 162.5)
- removed the D2 at (225.3, 162.5)
- removed the D2 at (150.3, 162.5)
- removed the D20 at (166.4, 182.3)
- removed the D20 at (316.4, 182.3)
- removed the D20 at (241.4, 182.3)
- removed the D21 at (330.4, 150.0)
- removed the D21 at (180.4, 150.0)
- removed the D21 at (255.4, 150.0)
- removed the D22 at (323.0, 160.4)
- removed the D22 at (248.0, 160.4)
- removed the D22 at (173.0, 160.4)
- removed the D23 at (234.9, 172.8)
- removed the D23 at (159.9, 172.8)
- removed the D23 at (309.9, 172.8)
- removed the D3 at (294.4, 155.2)
- removed the D3 at (219.3, 155.2)
- removed the D3 at (144.3, 155.2)
- removed the D4 at (219.3, 123.9)
- removed the D4 at (144.3, 123.9)
- removed the D4 at (294.3, 123.9)
- removed the D5 at (239.4, 171.7)
- removed the D5 at (164.4, 171.7)
- removed the D5 at (314.4, 171.7)
- removed the D6 at (147.0, 124.1)
- removed the D6 at (297.0, 124.1)
- removed the D6 at (222.0, 124.1)
- removed the D7 at (209.1, 169.2)
- removed the D7 at (284.1, 169.2)
- removed the D7 at (359.1, 169.2)
- removed the D8 at (150.1, 124.2)
- removed the D8 at (300.1, 124.2)
- removed the D8 at (225.1, 124.2)
- removed the D9 at (296.7, 148.5)
- removed the D9 at (221.7, 148.5)
- removed the D9 at (146.7, 148.5)
- removed the F1 at (309.5, 184.5)
- removed the F1 at (159.5, 184.5)
- removed the F1 at (234.5, 184.5)
- removed the FID1 at (141.0, 108.5)
- removed the FID1 at (291.0, 108.5)
- removed the FID1 at (216.0, 108.5)
- removed the FID1 at (66.0, 108.5)
- removed the FID2 at (66.0, 194.5)
- removed the FID2 at (216.0, 194.5)
- removed the FID2 at (291.0, 194.5)
- removed the FID2 at (141.0, 194.5)
- removed the FID3 at (362.0, 108.5)
- removed the FID3 at (137.0, 108.5)
- removed the FID3 at (212.0, 108.5)
- removed the FID3 at (287.0, 108.5)
- removed the FID4 at (212.0, 108.5)
- removed the FID4 at (362.0, 108.5)
- removed the FID4 at (137.0, 108.5)
- removed the FID4 at (287.0, 108.5)
- removed the FID5 at (291.0, 194.5)
- removed the FID5 at (216.0, 194.5)
- removed the FID5 at (141.0, 194.5)
- removed the FID6 at (141.0, 108.5)
- removed the FID6 at (291.0, 108.5)
- removed the FID6 at (216.0, 108.5)
- removed the J1 at (329.4, 153.6)
- removed the J1 at (179.4, 153.6)
- removed the J1 at (254.4, 153.6)
- removed the J10 at (359.9, 115.5)
- removed the J10 at (284.9, 115.5)
- removed the J10 at (209.9, 115.5)
- removed the J11 at (173.3, 115.8)
- removed the J11 at (323.4, 115.8)
- removed the J11 at (248.3, 115.8)
- removed the J2 at (357.6, 191.2)
- removed the J2 at (207.6, 191.2)
- removed the J2 at (282.6, 191.2)
- removed the J3 at (278.4, 184.7)
- removed the J3 at (203.3, 184.7)
- removed the J3 at (353.4, 184.7)
- removed the J4 at (188.0, 191.2)
- removed the J4 at (338.0, 191.2)
- removed the J4 at (263.0, 191.2)
- removed the J5 at (197.2, 191.3)
- removed the J5 at (347.2, 191.3)
- removed the J5 at (272.2, 191.3)
- removed the J6 at (359.8, 119.7)
- removed the J6 at (209.8, 119.7)
- removed the J6 at (284.8, 119.7)
- removed the J7 at (331.8, 182.5)
- removed the J7 at (256.8, 182.5)
- removed the J7 at (181.8, 182.5)
- removed the J9 at (236.0, 118.6)
- removed the J9 at (161.0, 118.6)
- removed the J9 at (311.0, 118.6)
- removed the JP1 at (248.7, 155.0)
- removed the JP1 at (173.7, 155.0)
- removed the JP1 at (323.7, 155.0)
- removed the K2 at (298.8, 166.4)
- removed the K2 at (148.8, 166.4)
- removed the K2 at (223.8, 166.4)
- removed the K3 at (300.1, 178.3)
- removed the K3 at (225.2, 178.3)
- removed the K3 at (150.2, 178.3)
- removed the L1 at (203.1, 156.6)
- removed the L1 at (353.1, 156.6)
- removed the L1 at (278.1, 156.6)
- removed the L2 at (315.4, 151.2)
- removed the L2 at (165.4, 151.2)
- removed the L2 at (240.4, 151.2)
- removed the L5 at (348.8, 186.2)
- removed the L5 at (198.8, 186.2)
- removed the L5 at (273.8, 186.2)
- removed the Q1 at (178.7, 160.6)
- removed the Q1 at (328.7, 160.6)
- removed the Q1 at (253.7, 160.6)
- removed the Q2 at (346.8, 139.6)
- removed the Q2 at (196.8, 139.6)
- removed the Q2 at (271.8, 139.6)
- removed the Q3 at (309.9, 173.6)
- removed the Q3 at (234.9, 173.6)
- removed the Q3 at (159.9, 173.6)
- removed the Q4 at (333.8, 158.2)
- removed the Q4 at (258.8, 158.2)
- removed the Q4 at (183.8, 158.2)
- removed the Q5 at (332.9, 136.5)
- removed the Q5 at (182.9, 136.5)
- removed the Q5 at (257.9, 136.5)
- removed the R10 at (197.2, 133.7)
- removed the R10 at (272.1, 133.7)
- removed the R10 at (347.1, 133.7)
- removed the R11 at (197.2, 129.4)
- removed the R11 at (272.2, 129.4)
- removed the R11 at (347.2, 129.4)
- removed the R12 at (200.4, 127.5)
- removed the R12 at (275.4, 127.5)
- removed the R12 at (350.4, 127.5)
- removed the R13 at (202.2, 127.5)
- removed the R13 at (277.1, 127.5)
- removed the R13 at (352.1, 127.5)
- removed the R14 at (145.0, 131.1)
- removed the R14 at (220.0, 131.1)
- removed the R14 at (295.0, 131.1)
- removed the R15 at (267.6, 157.4)
- removed the R15 at (192.6, 157.4)
- removed the R15 at (342.6, 157.4)
- removed the R16 at (347.1, 135.9)
- removed the R16 at (197.2, 135.9)
- removed the R16 at (272.1, 135.9)
- removed the R17 at (337.3, 157.4)
- removed the R17 at (187.3, 157.4)
- removed the R17 at (262.3, 157.4)
- removed the R18 at (133.1, 181.1)
- removed the R18 at (208.1, 181.1)
- removed the R18 at (358.1, 181.1)
- removed the R18 at (283.1, 181.1)
- removed the R19 at (280.4, 181.1)
- removed the R19 at (205.4, 181.1)
- removed the R19 at (130.4, 181.1)
- removed the R19 at (355.4, 181.1)
- removed the R20 at (248.1, 119.6)
- removed the R20 at (173.1, 119.6)
- removed the R20 at (323.1, 119.6)
- removed the R21 at (133.8, 178.1)
- removed the R21 at (208.8, 178.1)
- removed the R21 at (283.8, 178.1)
- removed the R21 at (358.8, 178.1)
- removed the R22 at (347.4, 153.1)
- removed the R22 at (272.4, 153.1)
- removed the R22 at (197.4, 153.1)
- removed the R23 at (279.0, 151.8)
- removed the R23 at (204.0, 151.8)
- removed the R23 at (354.0, 151.8)
- removed the R24 at (323.2, 121.6)
- removed the R24 at (173.2, 121.6)
- removed the R24 at (248.2, 121.6)
- removed the R25 at (348.3, 160.2)
- removed the R25 at (198.3, 160.2)
- removed the R25 at (273.3, 160.2)
- removed the R26 at (269.4, 160.2)
- removed the R26 at (194.4, 160.2)
- removed the R26 at (344.4, 160.2)
- removed the R27 at (206.4, 161.8)
- removed the R27 at (281.4, 161.8)
- removed the R27 at (356.4, 161.8)
- removed the R28 at (255.5, 148.2)
- removed the R28 at (330.5, 148.2)
- removed the R28 at (180.5, 148.2)
- removed the R29 at (330.4, 150.7)
- removed the R29 at (180.4, 150.7)
- removed the R29 at (255.4, 150.7)
- removed the R3 at (314.6, 184.2)
- removed the R3 at (239.7, 184.2)
- removed the R3 at (164.7, 184.2)
- removed the R30 at (337.9, 134.0)
- removed the R30 at (187.9, 134.0)
- removed the R30 at (262.9, 134.0)
- removed the R31 at (351.7, 147.2)
- removed the R31 at (201.7, 147.2)
- removed the R31 at (276.7, 147.2)
- removed the R32 at (206.8, 143.6)
- removed the R32 at (356.8, 143.6)
- removed the R32 at (281.8, 143.6)
- removed the R33 at (257.8, 139.6)
- removed the R33 at (332.8, 139.6)
- removed the R33 at (182.8, 139.6)
- removed the R34 at (280.6, 166.3)
- removed the R34 at (205.6, 166.3)
- removed the R34 at (355.6, 166.3)
- removed the R35 at (280.6, 168.4)
- removed the R35 at (355.6, 168.4)
- removed the R35 at (205.6, 168.4)
- removed the R36 at (313.3, 134.8)
- removed the R36 at (163.3, 134.8)
- removed the R36 at (238.3, 134.8)
- removed the R37 at (234.9, 161.0)
- removed the R37 at (309.9, 161.0)
- removed the R37 at (159.9, 161.0)
- removed the R38 at (313.6, 155.1)
- removed the R38 at (238.6, 155.1)
- removed the R38 at (163.6, 155.1)
- removed the R39 at (234.7, 168.8)
- removed the R39 at (309.7, 168.8)
- removed the R39 at (159.7, 168.8)
- removed the R4 at (167.5, 184.3)
- removed the R4 at (242.5, 184.3)
- removed the R4 at (317.5, 184.3)
- removed the R40 at (313.6, 152.8)
- removed the R40 at (163.6, 152.8)
- removed the R40 at (238.6, 152.8)
- removed the R41 at (148.2, 155.3)
- removed the R41 at (223.2, 155.3)
- removed the R41 at (298.2, 155.3)
- removed the R42 at (148.2, 157.9)
- removed the R42 at (298.2, 157.9)
- removed the R42 at (223.2, 157.9)
- removed the R43 at (182.3, 140.2)
- removed the R43 at (332.3, 140.2)
- removed the R43 at (257.3, 140.2)
- removed the R44 at (186.4, 140.1)
- removed the R44 at (261.4, 140.1)
- removed the R44 at (336.4, 140.1)
- removed the R45 at (206.5, 164.0)
- removed the R45 at (281.5, 164.0)
- removed the R45 at (356.5, 164.0)
- removed the R47 at (176.3, 155.2)
- removed the R47 at (251.3, 155.2)
- removed the R47 at (326.3, 155.2)
- removed the R49 at (176.3, 151.7)
- removed the R49 at (251.3, 151.7)
- removed the R49 at (326.3, 151.7)
- removed the R5 at (295.0, 129.2)
- removed the R5 at (220.0, 129.2)
- removed the R5 at (145.0, 129.2)
- removed the R50 at (172.6, 146.9)
- removed the R50 at (247.6, 146.9)
- removed the R50 at (322.6, 146.9)
- removed the R51 at (317.1, 152.8)
- removed the R51 at (242.1, 152.8)
- removed the R51 at (167.1, 152.8)
- removed the R52 at (175.2, 146.9)
- removed the R52 at (250.2, 146.9)
- removed the R52 at (325.2, 146.9)
- removed the R53 at (170.3, 146.8)
- removed the R53 at (245.3, 146.8)
- removed the R53 at (320.3, 146.8)
- removed the R54 at (350.3, 181.6)
- removed the R54 at (275.3, 181.6)
- removed the R54 at (200.3, 181.6)
- removed the R6 at (220.0, 127.5)
- removed the R6 at (295.0, 127.5)
- removed the R6 at (145.0, 127.5)
- removed the R7 at (220.1, 125.7)
- removed the R7 at (295.1, 125.7)
- removed the R7 at (145.1, 125.7)
- removed the R8 at (359.2, 157.0)
- removed the R8 at (209.2, 157.0)
- removed the R8 at (284.2, 157.0)
- removed the R9 at (284.2, 154.4)
- removed the R9 at (209.2, 154.4)
- removed the R9 at (359.2, 154.4)
- removed the TP4 at (173.2, 159.1)
- removed the TP4 at (323.2, 159.1)
- removed the TP4 at (248.2, 159.1)
- removed the U11 at (322.1, 152.9)
- removed the U11 at (247.1, 152.9)
- removed the U11 at (172.1, 152.9)
- removed the U12 at (306.1, 157.2)
- removed the U12 at (156.1, 157.2)
- removed the U12 at (231.1, 157.2)
- removed the U13 at (248.0, 130.6)
- removed the U13 at (173.0, 130.6)
- removed the U13 at (323.0, 130.6)
- removed the U14 at (188.2, 177.0)
- removed the U14 at (263.2, 177.0)
- removed the U14 at (338.2, 177.0)
- removed the U2 at (222.5, 156.2)
- removed the U2 at (147.5, 156.2)
- removed the U2 at (297.5, 156.2)
- removed the U3 at (336.6, 153.0)
- removed the U3 at (261.6, 153.0)
- removed the U3 at (186.7, 153.0)
- removed the U4 at (146.5, 134.7)
- removed the U4 at (221.5, 134.7)
- removed the U4 at (296.5, 134.7)
- removed the U5 at (342.8, 153.6)
- removed the U5 at (192.8, 153.6)
- removed the U5 at (267.8, 153.6)
- removed the U6 at (349.0, 132.3)
- removed the U6 at (274.0, 132.3)
- removed the U6 at (199.0, 132.3)
- removed the U7 at (268.8, 155.4)
- removed the U7 at (193.8, 155.4)
- removed the U7 at (343.8, 155.4)
- removed the U8 at (193.8, 172.8)
- removed the U8 at (268.8, 172.8)
- removed the U8 at (343.8, 172.8)
- removed the U9 at (164.9, 163.7)
- removed the U9 at (314.9, 163.7)
- removed the U9 at (239.9, 163.7)
- removed the Y1 at (266.7, 145.4)
- removed the Y1 at (341.7, 145.4)
- removed the Y1 at (191.7, 145.4)
- removed the Y4 at (169.0, 142.6)
- removed the Y4 at (319.0, 142.6)
- removed the Y4 at (244.0, 142.6)
- removed the Y5 at (175.3, 144.0)
- removed the Y5 at (250.3, 144.0)
- removed the Y5 at (325.3, 144.0)
- added 3.3V1: 3.3V, TestPoint:TestPoint_Pad_1.0x1.0mm, F.Cu at (154.9, 128.7)
- added 3.3V2: 3.3V, TestPoint:TestPoint_Pad_1.0x1.0mm, F.Cu at (229.9, 128.7)
- added 3.3V3: 3.3V, TestPoint:TestPoint_Pad_1.0x1.0mm, F.Cu at (304.9, 128.7)
- added 5V1: 5V, TestPoint:TestPoint_Pad_1.0x1.0mm, F.Cu at (154.2, 119.8)
- added 5V2: 5V, TestPoint:TestPoint_Pad_1.0x1.0mm, F.Cu at (229.2, 119.8)
- added 5V3: 5V, TestPoint:TestPoint_Pad_1.0x1.0mm, F.Cu at (304.2, 119.8)
- added BT2: 1056, 1056:BAT_1056, B.Cu at (187.3, 124.5)
- added BT3: 1056, 1056:BAT_1056, B.Cu at (262.3, 124.5)
- added BT4: 1056, 1056:BAT_1056, B.Cu at (337.3, 124.5)
- added BZ2: Buzzer, Buzzer_Beeper:MagneticBuzzer_ProSignal_ABI-009-RC, F.Cu at (191.4, 122.8)
- added BZ3: Buzzer, Buzzer_Beeper:MagneticBuzzer_ProSignal_ABI-009-RC, F.Cu at (266.4, 122.8)
- added BZ4: Buzzer, Buzzer_Beeper:MagneticBuzzer_ProSignal_ABI-009-RC, F.Cu at (341.4, 122.8)
- added C100: 10uF/25V, Capacitor_THT:CP_Radial_D5.0mm_P2.50mm, F.Cu at (231.7, 142.0)
- added C101: 10uF/25V, Capacitor_THT:CP_Radial_D5.0mm_P2.50mm, F.Cu at (229.8, 136.0)
- added C102: 1uF/16V, Capacitor_SMD:C_0603_1608Metric, B.Cu at (230.5, 139.2)
- added C103: 0.1uF/16V, Capacitor_SMD:C_0603_1608Metric, F.Cu at (282.6, 151.8)
- added C104: 100uFx6.3v, Capacitor_SMD:C_Elec_5x5.8, F.Cu at (249.0, 183.0)
- added C105: 220uF/10v, Capacitor_SMD:CP_Elec_8x6.5, F.Cu at (247.4, 174.2)
- added C106: 0.1uFx/10V, Capacitor_SMD:C_0805_2012Metric, F.Cu at (248.0, 165.4)
- added C107: 1uF, Capacitor_SMD:C_0603_1608Metric, F.Cu at (261.9, 144.2)
- added C108: 18pF, Capacitor_SMD:C_0603_1608Metric, F.Cu at (268.0, 141.5)
- added C109: 18pF, Capacitor_SMD:C_0603_1608Metric, F.Cu at (271.8, 141.6)
- added C110: 1uF/6.3V, Capacitor_SMD:C_0603_1608Metric, F.Cu at (253.9, 119.9)
- added C111: 0.1uF/6.3V, Capacitor_SMD:C_0603_1608Metric, F.Cu at (253.9, 121.7)
- added C112: 1uF/6.3V, Capacitor_SMD:C_0603_1608Metric, F.Cu at (244.9, 121.6)
- added C113: 0.1uF/6.3V, Capacitor_SMD:C_0603_1608Metric, F.Cu at (244.8, 119.7)
- added C114: 1uF/6.3V, Capacitor_SMD:C_0603_1608Metric, F.Cu at (239.1, 140.5)
- added C115: 0.1uF/6.3V, Capacitor_SMD:C_0603_1608Metric, F.Cu at (238.3, 136.6)
- added C116: 1uF/6.3V, Capacitor_SMD:C_0603_1608Metric, F.Cu at (257.7, 135.6)
- added C117: 0.1uF/6.3V, Capacitor_SMD:C_0603_1608Metric, F.Cu at (259.6, 135.7)
- added C118: 0.1uFx/10V, Capacitor_SMD:C_0805_2012Metric, F.Cu at (253.5, 168.0)
- added C119: 1uF/6.3V, Capacitor_SMD:C_0603_1608Metric, F.Cu at (262.1, 131.6)
- added C120: 0.1uF/6.3V, Capacitor_SMD:C_0603_1608Metric, F.Cu at (263.7, 131.6)
- added C121: 1uF/6.3V, Capacitor_SMD:C_0603_1608Metric, F.Cu at (282.8, 129.3)
- added C122: 0.1uF/6.3V, Capacitor_SMD:C_0603_1608Metric, F.Cu at (284.9, 129.3)
- added C123: 0.1uF, Capacitor_SMD:C_0603_1608Metric, B.Cu at (238.5, 157.1)
- added C124: 0.1uF, Capacitor_SMD:C_0603_1608Metric, B.Cu at (248.3, 165.8)
- added C125: 0.1uF, Capacitor_SMD:C_0603_1608Metric, B.Cu at (245.6, 166.7)
- added C126: 0.1uF, Capacitor_SMD:C_0603_1608Metric, B.Cu at (242.0, 157.1)
- added C127: 0.1uF, Capacitor_SMD:C_0603_1608Metric, B.Cu at (242.0, 155.2)
- added C128: 22pF, Capacitor_SMD:C_0603_1608Metric, F.Cu at (245.3, 140.3)
- added C129: 330uF, Capacitor_Tantalum_SMD:CP_EIA-6032-15_Kemet-U, F.Cu at (254.0, 173.2)
- added C130: 10uFx/10V, Capacitor_SMD:C_0603_1608Metric, F.Cu at (253.6, 165.1)
- added C131: 22pF, Capacitor_SMD:C_0603_1608Metric, F.Cu at (242.2, 140.3)
- added C132: 18pF, Capacitor_SMD:C_0603_1608Metric, F.Cu at (248.4, 140.3)
- added C133: 18pF, Capacitor_SMD:C_0603_1608Metric, F.Cu at (251.5, 140.3)
- added C134: 1uF/6.3V, Capacitor_SMD:C_0603_1608Metric, F.Cu at (279.1, 147.2)
- added C135: 0.1uF/6.3V, Capacitor_SMD:C_0603_1608Metric, F.Cu at (281.8, 147.2)
- added C136: 1uF/6.3V, Capacitor_SMD:C_0603_1608Metric, F.Cu at (262.9, 135.8)
- added C137: 0.1uF/6.3V, Capacitor_SMD:C_0603_1608Metric, F.Cu at (262.9, 137.7)
- added C138: 1uF, Capacitor_SMD:C_0603_1608Metric, B.Cu at (248.1, 162.3)
- added C139: 220uF/25V, Capacitor_SMD:CP_Elec_8x6.9, F.Cu at (313.7, 163.1)
- added C140: 10uFx16v, Capacitor_SMD:C_0603_1608Metric, B.Cu at (355.5, 164.3)
- added C141: 220uF/25V, Capacitor_SMD:CP_Elec_8x6.9, F.Cu at (297.9, 143.6)
- added C142: 1uF, Capacitor_SMD:C_0603_1608Metric, B.Cu at (312.3, 139.3)
- added C143: 1uF, Capacitor_SMD:C_0603_1608Metric, F.Cu at (307.0, 149.0)
- added C144: 10uF/16V, Capacitor_SMD:C_0603_1608Metric, F.Cu at (359.3, 159.4)
- added C145: 10uF/16V, Capacitor_SMD:C_0603_1608Metric, F.Cu at (360.0, 163.0)
- added C146: 10uF/25V, Capacitor_THT:CP_Radial_D5.0mm_P2.50mm, F.Cu at (306.7, 142.0)
- added C147: 10uF/25V, Capacitor_THT:CP_Radial_D5.0mm_P2.50mm, F.Cu at (304.8, 136.0)
- added C148: 1uF/16V, Capacitor_SMD:C_0603_1608Metric, B.Cu at (305.5, 139.2)
- added C149: 0.1uF/16V, Capacitor_SMD:C_0603_1608Metric, F.Cu at (357.6, 151.8)
- added C150: 100uFx6.3v, Capacitor_SMD:C_Elec_5x5.8, F.Cu at (324.0, 183.0)
- added C151: 220uF/10v, Capacitor_SMD:CP_Elec_8x6.5, F.Cu at (322.4, 174.2)
- added C152: 0.1uFx/10V, Capacitor_SMD:C_0805_2012Metric, F.Cu at (323.0, 165.4)
- added C153: 1uF, Capacitor_SMD:C_0603_1608Metric, F.Cu at (336.9, 144.2)
- added C154: 18pF, Capacitor_SMD:C_0603_1608Metric, F.Cu at (343.0, 141.5)
- added C155: 18pF, Capacitor_SMD:C_0603_1608Metric, F.Cu at (346.8, 141.6)
- added C156: 1uF/6.3V, Capacitor_SMD:C_0603_1608Metric, F.Cu at (328.9, 119.9)
- added C157: 0.1uF/6.3V, Capacitor_SMD:C_0603_1608Metric, F.Cu at (328.9, 121.7)
- added C158: 1uF/6.3V, Capacitor_SMD:C_0603_1608Metric, F.Cu at (319.9, 121.6)
- added C159: 0.1uF/6.3V, Capacitor_SMD:C_0603_1608Metric, F.Cu at (319.8, 119.7)
- added C160: 1uF/6.3V, Capacitor_SMD:C_0603_1608Metric, F.Cu at (314.1, 140.5)
- added C161: 0.1uF/6.3V, Capacitor_SMD:C_0603_1608Metric, F.Cu at (313.3, 136.6)
- added C162: 1uF/6.3V, Capacitor_SMD:C_0603_1608Metric, F.Cu at (332.7, 135.6)
- added C163: 0.1uF/6.3V, Capacitor_SMD:C_0603_1608Metric, F.Cu at (334.6, 135.7)
- added C164: 0.1uFx/10V, Capacitor_SMD:C_0805_2012Metric, F.Cu at (328.5, 168.0)
- added C165: 1uF/6.3V, Capacitor_SMD:C_0603_1608Metric, F.Cu at (337.1, 131.6)
- added C166: 0.1uF/6.3V, Capacitor_SMD:C_0603_1608Metric, F.Cu at (338.7, 131.6)
- added C167: 1uF/6.3V, Capacitor_SMD:C_0603_1608Metric, F.Cu at (357.8, 129.3)
- added C168: 0.1uF/6.3V, Capacitor_SMD:C_0603_1608Metric, F.Cu at (359.9, 129.3)
- added C169: 0.1uF, Capacitor_SMD:C_0603_1608Metric, B.Cu at (313.5, 157.1)
- added C170: 0.1uF, Capacitor_SMD:C_0603_1608Metric, B.Cu at (323.3, 165.8)
- added C171: 0.1uF, Capacitor_SMD:C_0603_1608Metric, B.Cu at (320.6, 166.7)
- added C172: 0.1uF, Capacitor_SMD:C_0603_1608Metric, B.Cu at (317.0, 157.1)
- added C173: 0.1uF, Capacitor_SMD:C_0603_1608Metric, B.Cu at (317.0, 155.2)
- added C174: 22pF, Capacitor_SMD:C_0603_1608Metric, F.Cu at (320.3, 140.3)
- added C175: 330uF, Capacitor_Tantalum_SMD:CP_EIA-6032-15_Kemet-U, F.Cu at (329.0, 173.2)
- added C176: 10uFx/10V, Capacitor_SMD:C_0603_1608Metric, F.Cu at (328.6, 165.1)
- added C177: 22pF, Capacitor_SMD:C_0603_1608Metric, F.Cu at (317.2, 140.3)
- added C178: 18pF, Capacitor_SMD:C_0603_1608Metric, F.Cu at (323.4, 140.3)
- added C179: 18pF, Capacitor_SMD:C_0603_1608Metric, F.Cu at (326.5, 140.3)
- added C180: 1uF/6.3V, Capacitor_SMD:C_0603_1608Metric, F.Cu at (354.1, 147.2)
- added C181: 0.1uF/6.3V, Capacitor_SMD:C_0603_1608Metric, F.Cu at (356.8, 147.2)
- added C182: 1uF/6.3V, Capacitor_SMD:C_0603_1608Metric, F.Cu at (337.9, 135.8)
- added C183: 0.1uF/6.3V, Capacitor_SMD:C_0603_1608Metric, F.Cu at (337.9, 137.7)
- added C184: 1uF, Capacitor_SMD:C_0603_1608Metric, B.Cu at (323.1, 162.3)
- added C3: 220uF/25V, Capacitor_SMD:CP_Elec_8x6.9, F.Cu at (163.7, 163.1)
- added C48: 10uFx16v, Capacitor_SMD:C_0603_1608Metric, B.Cu at (205.5, 164.3)
- added C49: 220uF/25V, Capacitor_SMD:CP_Elec_8x6.9, F.Cu at (147.9, 143.6)
- added C50: 1uF, Capacitor_SMD:C_0603_1608Metric, B.Cu at (162.3, 139.3)
- added C51: 1uF, Capacitor_SMD:C_0603_1608Metric, F.Cu at (157.0, 149.0)
- added C52: 10uF/16V, Capacitor_SMD:C_0603_1608Metric, F.Cu at (209.3, 159.4)
- added C53: 10uF/16V, Capacitor_SMD:C_0603_1608Metric, F.Cu at (210.0, 163.0)
- added C54: 10uF/25V, Capacitor_THT:CP_Radial_D5.0mm_P2.50mm, F.Cu at (156.7, 142.0)
- added C55: 10uF/25V, Capacitor_THT:CP_Radial_D5.0mm_P2.50mm, F.Cu at (154.8, 136.0)
- added C56: 1uF/16V, Capacitor_SMD:C_0603_1608Metric, B.Cu at (155.5, 139.2)
- added C57: 0.1uF/16V, Capacitor_SMD:C_0603_1608Metric, F.Cu at (207.6, 151.8)
- added C58: 100uFx6.3v, Capacitor_SMD:C_Elec_5x5.8, F.Cu at (174.0, 183.0)
- added C59: 220uF/10v, Capacitor_SMD:CP_Elec_8x6.5, F.Cu at (172.4, 174.2)
- added C60: 0.1uFx/10V, Capacitor_SMD:C_0805_2012Metric, F.Cu at (173.0, 165.4)
- added C61: 1uF, Capacitor_SMD:C_0603_1608Metric, F.Cu at (186.9, 144.2)
- added C62: 18pF, Capacitor_SMD:C_0603_1608Metric, F.Cu at (193.0, 141.5)
- added C63: 18pF, Capacitor_SMD:C_0603_1608Metric, F.Cu at (196.8, 141.6)
- added C64: 1uF/6.3V, Capacitor_SMD:C_0603_1608Metric, F.Cu at (178.9, 119.9)
- added C65: 0.1uF/6.3V, Capacitor_SMD:C_0603_1608Metric, F.Cu at (178.9, 121.7)
- added C66: 1uF/6.3V, Capacitor_SMD:C_0603_1608Metric, F.Cu at (169.9, 121.6)
- added C67: 0.1uF/6.3V, Capacitor_SMD:C_0603_1608Metric, F.Cu at (169.8, 119.7)
- added C68: 1uF/6.3V, Capacitor_SMD:C_0603_1608Metric, F.Cu at (164.1, 140.5)
- added C69: 0.1uF/6.3V, Capacitor_SMD:C_0603_1608Metric, F.Cu at (163.3, 136.6)
- added C70: 1uF/6.3V, Capacitor_SMD:C_0603_1608Metric, F.Cu at (182.7, 135.6)
- added C71: 0.1uF/6.3V, Capacitor_SMD:C_0603_1608Metric, F.Cu at (184.6, 135.7)
- added C72: 0.1uFx/10V, Capacitor_SMD:C_0805_2012Metric, F.Cu at (178.5, 168.0)
- added C73: 1uF/6.3V, Capacitor_SMD:C_0603_1608Metric, F.Cu at (187.1, 131.6)
- added C74: 0.1uF/6.3V, Capacitor_SMD:C_0603_1608Metric, F.Cu at (188.7, 131.6)
- added C75: 1uF/6.3V, Capacitor_SMD:C_0603_1608Metric, F.Cu at (207.8, 129.3)
- added C76: 0.1uF/6.3V, Capacitor_SMD:C_0603_1608Metric, F.Cu at (209.9, 129.3)
- added C77: 0.1uF, Capacitor_SMD:C_0603_1608Metric, B.Cu at (163.5, 157.1)
- added C78: 0.1uF, Capacitor_SMD:C_0603_1608Metric, B.Cu at (173.3, 165.8)
- added C79: 0.1uF, Capacitor_SMD:C_0603_1608Metric, B.Cu at (170.6, 166.7)
- added C80: 0.1uF, Capacitor_SMD:C_0603_1608Metric, B.Cu at (167.0, 157.1)
- added C81: 0.1uF, Capacitor_SMD:C_0603_1608Metric, B.Cu at (167.0, 155.2)
- added C82: 22pF, Capacitor_SMD:C_0603_1608Metric, F.Cu at (170.3, 140.3)
- added C83: 330uF, Capacitor_Tantalum_SMD:CP_EIA-6032-15_Kemet-U, F.Cu at (179.0, 173.2)
- added C84: 10uFx/10V, Capacitor_SMD:C_0603_1608Metric, F.Cu at (178.6, 165.1)
- added C85: 22pF, Capacitor_SMD:C_0603_1608Metric, F.Cu at (167.2, 140.3)
- added C86: 18pF, Capacitor_SMD:C_0603_1608Metric, F.Cu at (173.4, 140.3)
- added C87: 18pF, Capacitor_SMD:C_0603_1608Metric, F.Cu at (176.5, 140.3)
- added C88: 1uF/6.3V, Capacitor_SMD:C_0603_1608Metric, F.Cu at (204.2, 147.2)
- added C89: 0.1uF/6.3V, Capacitor_SMD:C_0603_1608Metric, F.Cu at (206.8, 147.2)
- added C90: 1uF/6.3V, Capacitor_SMD:C_0603_1608Metric, F.Cu at (187.9, 135.8)
- added C91: 0.1uF/6.3V, Capacitor_SMD:C_0603_1608Metric, F.Cu at (187.9, 137.7)
- added C92: 1uF, Capacitor_SMD:C_0603_1608Metric, B.Cu at (173.1, 162.3)
- added C93: 220uF/25V, Capacitor_SMD:CP_Elec_8x6.9, F.Cu at (238.7, 163.1)
- added C94: 10uFx16v, Capacitor_SMD:C_0603_1608Metric, B.Cu at (280.5, 164.3)
- added C95: 220uF/25V, Capacitor_SMD:CP_Elec_8x6.9, F.Cu at (222.9, 143.6)
- added C96: 1uF, Capacitor_SMD:C_0603_1608Metric, B.Cu at (237.3, 139.3)
- added C97: 1uF, Capacitor_SMD:C_0603_1608Metric, F.Cu at (232.0, 149.0)
- added C98: 10uF/16V, Capacitor_SMD:C_0603_1608Metric, F.Cu at (284.3, 159.4)
- added C99: 10uF/16V, Capacitor_SMD:C_0603_1608Metric, F.Cu at (285.0, 163.0)
- added CN2: Main_Connector, 66201821122:66201821122, F.Cu at (167.9, 190.6)
- added CN3: Main_Connector, 66201821122:66201821122, F.Cu at (242.9, 190.6)
- added CN4: Main_Connector, 66201821122:66201821122, F.Cu at (317.9, 190.6)
- added D14: Schottkey, Diode_SMD:D_SOD-123, B.Cu at (134.1, 179.6)
- added D24: 3.9 Zener, Diode_SMD:D_SOD-123, F.Cu at (164.7, 178.4)
- added D25: Schottkey/1A, Diode_SMD:D_SMA, B.Cu at (150.3, 162.5)
- added D26: Schottkey/1A, Diode_SMD:D_SMA, B.Cu at (144.3, 155.2)
- added D27: R_LED, LED_SMD:LED_0805_2012Metric, F.Cu at (144.3, 123.9)
- added D28: Schottkey/1A, Diode_SMD:D_SMA, F.Cu at (164.4, 171.7)
- added D29: G_LED, LED_SMD:LED_0805_2012Metric, F.Cu at (147.0, 124.1)
- added D30: Schottkey/1A, Diode_SMD:D_SMA, B.Cu at (209.1, 169.2)
- added D31: GPRS_LED, LED_SMD:LED_0805_2012Metric, F.Cu at (150.1, 124.2)
- added D32: G_Purpose, Diode_SMD:D_SMA, B.Cu at (146.7, 148.5)
- added D33: 3.9 Zener, Diode_SMD:D_SOD-123, B.Cu at (198.0, 131.5)
- added D34: 3.9 Zener, Diode_SMD:D_SOD-123, B.Cu at (204.1, 128.3)
- added D35: PW_LED, LED_SMD:LED_0805_2012Metric, F.Cu at (145.1, 128.3)
- added D36: Power, LED_SMD:LED_0805_2012Metric, F.Cu at (196.9, 156.2)
- added D37: Schottkey, Diode_SMD:D_SOD-123, B.Cu at (209.1, 179.6)
- added D38: 3.9 Zener, Diode_SMD:D_SOD-123, F.Cu at (165.8, 121.2)
- added D39: G_purpose, Diode_SMD:D_SMA, B.Cu at (178.4, 162.7)
- added D40: ST, LED_SMD:LED_0805_2012Metric, F.Cu at (208.8, 173.3)
- added D41: NW, LED_SMD:LED_0805_2012Metric, F.Cu at (208.7, 170.3)
- added D42: 1N4148, Diode_SMD:D_SOD-123, F.Cu at (161.9, 139.9)
- added D43: G_Purpose, Diode_SMD:D_SMA, B.Cu at (166.4, 182.3)
- added D44: 3.9 Zener, Diode_SMD:D_SOD-123, B.Cu at (180.4, 150.0)
- added D45: 3.9 Zener, Diode_SMD:D_SOD-123, F.Cu at (173.0, 160.4)
- added D46: ?, Diode_SMD:D_SMA, B.Cu at (159.9, 172.8)
- added D47: 3.9 Zener, Diode_SMD:D_SOD-123, F.Cu at (239.7, 178.4)
- added D48: Schottkey/1A, Diode_SMD:D_SMA, B.Cu at (225.3, 162.5)
- added D49: Schottkey/1A, Diode_SMD:D_SMA, B.Cu at (219.3, 155.2)
- added D50: R_LED, LED_SMD:LED_0805_2012Metric, F.Cu at (219.3, 123.9)
- added D51: Schottkey/1A, Diode_SMD:D_SMA, F.Cu at (239.4, 171.7)
- added D52: G_LED, LED_SMD:LED_0805_2012Metric, F.Cu at (222.0, 124.1)
- added D53: Schottkey/1A, Diode_SMD:D_SMA, B.Cu at (284.1, 169.2)
- added D54: GPRS_LED, LED_SMD:LED_0805_2012Metric, F.Cu at (225.1, 124.2)
- added D55: G_Purpose, Diode_SMD:D_SMA, B.Cu at (221.7, 148.5)
- added D56: 3.9 Zener, Diode_SMD:D_SOD-123, B.Cu at (273.0, 131.5)
- added D57: 3.9 Zener, Diode_SMD:D_SOD-123, B.Cu at (279.1, 128.3)
- added D58: PW_LED, LED_SMD:LED_0805_2012Metric, F.Cu at (220.1, 128.3)
- added D59: Power, LED_SMD:LED_0805_2012Metric, F.Cu at (271.9, 156.2)
- added D60: Schottkey, Diode_SMD:D_SOD-123, B.Cu at (284.1, 179.6)
- added D61: 3.9 Zener, Diode_SMD:D_SOD-123, F.Cu at (240.8, 121.2)
- added D62: G_purpose, Diode_SMD:D_SMA, B.Cu at (253.4, 162.7)
- added D63: ST, LED_SMD:LED_0805_2012Metric, F.Cu at (283.8, 173.3)
- added D64: NW, LED_SMD:LED_0805_2012Metric, F.Cu at (283.7, 170.3)
- added D65: 1N4148, Diode_SMD:D_SOD-123, F.Cu at (236.9, 139.9)
- added D66: G_Purpose, Diode_SMD:D_SMA, B.Cu at (241.4, 182.3)
- added D67: 3.9 Zener, Diode_SMD:D_SOD-123, B.Cu at (255.4, 150.0)
- added D68: 3.9 Zener, Diode_SMD:D_SOD-123, F.Cu at (248.0, 160.4)
- added D69: ?, Diode_SMD:D_SMA, B.Cu at (234.9, 172.8)
- added D70: 3.9 Zener, Diode_SMD:D_SOD-123, F.Cu at (314.7, 178.4)
- added D71: Schottkey/1A, Diode_SMD:D_SMA, B.Cu at (300.3, 162.5)
- added D72: Schottkey/1A, Diode_SMD:D_SMA, B.Cu at (294.4, 155.2)
- added D73: R_LED, LED_SMD:LED_0805_2012Metric, F.Cu at (294.3, 123.9)
- added D74: Schottkey/1A, Diode_SMD:D_SMA, F.Cu at (314.4, 171.7)
- added D75: G_LED, LED_SMD:LED_0805_2012Metric, F.Cu at (297.0, 124.1)
- added D76: Schottkey/1A, Diode_SMD:D_SMA, B.Cu at (359.1, 169.2)
- added D77: GPRS_LED, LED_SMD:LED_0805_2012Metric, F.Cu at (300.1, 124.2)
- added D78: G_Purpose, Diode_SMD:D_SMA, B.Cu at (296.7, 148.5)
- added D79: 3.9 Zener, Diode_SMD:D_SOD-123, B.Cu at (348.0, 131.5)
- added D80: 3.9 Zener, Diode_SMD:D_SOD-123, B.Cu at (354.1, 128.3)
- added D81: PW_LED, LED_SMD:LED_0805_2012Metric, F.Cu at (295.1, 128.3)
- added D82: Power, LED_SMD:LED_0805_2012Metric, F.Cu at (346.9, 156.2)
- added D83: Schottkey, Diode_SMD:D_SOD-123, B.Cu at (359.1, 179.6)
- added D84: 3.9 Zener, Diode_SMD:D_SOD-123, F.Cu at (315.8, 121.2)
- added D85: G_purpose, Diode_SMD:D_SMA, B.Cu at (328.4, 162.7)
- added D86: ST, LED_SMD:LED_0805_2012Metric, F.Cu at (358.8, 173.3)
- added D87: NW, LED_SMD:LED_0805_2012Metric, F.Cu at (358.7, 170.3)
- added D88: 1N4148, Diode_SMD:D_SOD-123, F.Cu at (311.9, 139.9)
- added D89: G_Purpose, Diode_SMD:D_SMA, B.Cu at (316.4, 182.3)
- added D90: 3.9 Zener, Diode_SMD:D_SOD-123, B.Cu at (330.4, 150.0)
- added D91: 3.9 Zener, Diode_SMD:D_SOD-123, F.Cu at (323.0, 160.4)
- added D92: ?, Diode_SMD:D_SMA, B.Cu at (309.9, 172.8)
- added F2: 30V/0.09A, Fuse:Fuse_BelFuse_0ZRE0005FF_L8.3mm_W3.8mm, F.Cu at (159.5, 184.5)
- added F3: 30V/0.09A, Fuse:Fuse_BelFuse_0ZRE0005FF_L8.3mm_W3.8mm, F.Cu at (234.5, 184.5)
- added F4: 30V/0.09A, Fuse:Fuse_BelFuse_0ZRE0005FF_L8.3mm_W3.8mm, F.Cu at (309.5, 184.5)
- added FID1: Fiducial, Fiducial:Fiducial_1mm_Mask3mm, F.Cu at (66.0, 108.5)
- added FID10: Fiducial, Fiducial:Fiducial_1.5mm_Mask3mm, B.Cu at (212.0, 108.5)
- added FID11: Fiducial, Fiducial:Fiducial_0.75mm_Mask1.5mm, B.Cu at (141.0, 194.5)
- added FID12: Fiducial, Fiducial:Fiducial_0.75mm_Mask1.5mm, B.Cu at (141.0, 108.5)
- added FID13: Fiducial, Fiducial:Fiducial_1mm_Mask3mm, F.Cu at (216.0, 108.5)
- added FID14: Fiducial, Fiducial:Fiducial_1mm_Mask3mm, F.Cu at (216.0, 194.5)
- added FID15: Fiducial, Fiducial:Fiducial_1mm_Mask3mm, F.Cu at (287.0, 108.5)
- added FID16: Fiducial, Fiducial:Fiducial_1.5mm_Mask3mm, B.Cu at (287.0, 108.5)
- added FID17: Fiducial, Fiducial:Fiducial_0.75mm_Mask1.5mm, B.Cu at (216.0, 194.5)
- added FID18: Fiducial, Fiducial:Fiducial_0.75mm_Mask1.5mm, B.Cu at (216.0, 108.5)
- added FID19: Fiducial, Fiducial:Fiducial_1mm_Mask3mm, F.Cu at (291.0, 108.5)
- added FID2: Fiducial, Fiducial:Fiducial_1mm_Mask3mm, F.Cu at (66.0, 194.5)
- added FID20: Fiducial, Fiducial:Fiducial_1mm_Mask3mm, F.Cu at (291.0, 194.5)
- added FID21: Fiducial, Fiducial:Fiducial_1mm_Mask3mm, F.Cu at (362.0, 108.5)
- added FID22: Fiducial, Fiducial:Fiducial_1.5mm_Mask3mm, B.Cu at (362.0, 108.5)
- added FID23: Fiducial, Fiducial:Fiducial_0.75mm_Mask1.5mm, B.Cu at (291.0, 194.5)
- added FID24: Fiducial, Fiducial:Fiducial_0.75mm_Mask1.5mm, B.Cu at (291.0, 108.5)
- added FID3: Fiducial, Fiducial:Fiducial_1mm_Mask3mm, F.Cu at (137.0, 108.5)
- added FID4: Fiducial, Fiducial:Fiducial_1.5mm_Mask3mm, B.Cu at (137.0, 108.5)
- added FID7: Fiducial, Fiducial:Fiducial_1mm_Mask3mm, F.Cu at (141.0, 108.5)
- added FID8: Fiducial, Fiducial:Fiducial_1mm_Mask3mm, F.Cu at (141.0, 194.5)
- added FID9: Fiducial, Fiducial:Fiducial_1mm_Mask3mm, F.Cu at (212.0, 108.5)
- added J12: USB_B_Mini, Connector_USB:USB_Mini-B_Lumberg_2486_01_Horizontal, F.Cu at (207.6, 191.2)
- added J13: USB_Con, Connector_PinSocket_2.54mm:PinSocket_1x04_P2.54mm_Vertical, F.Cu at (203.3, 184.7)
- added J14: ANT, Connector_Coaxial:SMA_Amphenol_132291_Vertical, F.Cu at (188.0, 191.2)
- added J15: Conn_Coaxial, Connector_Coaxial:SMA_Amphenol_132291_Vertical, F.Cu at (197.2, 191.3)
- added J16: Debug/GPS_DBG, Connector_PinSocket_2.54mm:PinSocket_1x05_P2.54mm_Vertical, F.Cu at (209.8, 119.7)
- added J17: Conn_Coaxial, Connector_Coaxial:U.FL_Molex_MCRF_73412-0110_Vertical, F.Cu at (181.8, 182.5)
- added J18: Prog_G, Connector_PinSocket_2.54mm:PinSocket_1x06_P2.54mm_Vertical, F.Cu at (161.0, 118.6)
- added J19: Prog_T, Connector_PinSocket_2.54mm:PinSocket_1x06_P2.54mm_Vertical, F.Cu at (209.9, 115.5)
- added J20: Debug, Connector_PinHeader_2.54mm:PinHeader_1x03_P2.54mm_Vertical, F.Cu at (173.3, 115.8)
- added J21: Conn_01x02, Connector_JST:JST_PH_B2B-PH-K_1x02_P2.00mm_Vertical, B.Cu at (254.4, 153.6)
- added J22: USB_B_Mini, Connector_USB:USB_Mini-B_Lumberg_2486_01_Horizontal, F.Cu at (282.6, 191.2)
- added J23: USB_Con, Connector_PinSocket_2.54mm:PinSocket_1x04_P2.54mm_Vertical, F.Cu at (278.4, 184.7)
- added J24: ANT, Connector_Coaxial:SMA_Amphenol_132291_Vertical, F.Cu at (263.0, 191.2)
- added J25: Conn_Coaxial, Connector_Coaxial:SMA_Amphenol_132291_Vertical, F.Cu at (272.2, 191.3)
- added J26: Debug/GPS_DBG, Connector_PinSocket_2.54mm:PinSocket_1x05_P2.54mm_Vertical, F.Cu at (284.8, 119.7)
- added J27: Conn_Coaxial, Connector_Coaxial:U.FL_Molex_MCRF_73412-0110_Vertical, F.Cu at (256.8, 182.5)
- added J28: Prog_G, Connector_PinSocket_2.54mm:PinSocket_1x06_P2.54mm_Vertical, F.Cu at (236.0, 118.6)
- added J29: Prog_T, Connector_PinSocket_2.54mm:PinSocket_1x06_P2.54mm_Vertical, F.Cu at (284.9, 115.5)
- added J30: Debug, Connector_PinHeader_2.54mm:PinHeader_1x03_P2.54mm_Vertical, F.Cu at (248.3, 115.8)
- added J31: Conn_01x02, Connector_JST:JST_PH_B2B-PH-K_1x02_P2.00mm_Vertical, B.Cu at (329.4, 153.6)
- added J32: USB_B_Mini, Connector_USB:USB_Mini-B_Lumberg_2486_01_Horizontal, F.Cu at (357.6, 191.2)
- added J33: USB_Con, Connector_PinSocket_2.54mm:PinSocket_1x04_P2.54mm_Vertical, F.Cu at (353.4, 184.7)
- added J34: ANT, Connector_Coaxial:SMA_Amphenol_132291_Vertical, F.Cu at (338.0, 191.2)
- added J35: Conn_Coaxial, Connector_Coaxial:SMA_Amphenol_132291_Vertical, F.Cu at (347.2, 191.3)
- added J36: Debug/GPS_DBG, Connector_PinSocket_2.54mm:PinSocket_1x05_P2.54mm_Vertical, F.Cu at (359.8, 119.7)
- added J37: Conn_Coaxial, Connector_Coaxial:U.FL_Molex_MCRF_73412-0110_Vertical, F.Cu at (331.8, 182.5)
- added J38: Prog_G, Connector_PinSocket_2.54mm:PinSocket_1x06_P2.54mm_Vertical, F.Cu at (311.0, 118.6)
- added J39: Prog_T, Connector_PinSocket_2.54mm:PinSocket_1x06_P2.54mm_Vertical, F.Cu at (359.9, 115.5)
- added J40: Debug, Connector_PinHeader_2.54mm:PinHeader_1x03_P2.54mm_Vertical, F.Cu at (323.4, 115.8)
- added J8: Conn_01x02, Connector_JST:JST_PH_B2B-PH-K_1x02_P2.00mm_Vertical, B.Cu at (179.4, 153.6)
- added JP2: Analog fuel jumper, Jumper:SolderJumper-2_P1.3mm_Open_RoundedPad1.0x1.5mm, F.Cu at (173.7, 155.0)
- added JP3: Analog fuel jumper, Jumper:SolderJumper-2_P1.3mm_Open_RoundedPad1.0x1.5mm, F.Cu at (248.7, 155.0)
- added JP4: Analog fuel jumper, Jumper:SolderJumper-2_P1.3mm_Open_RoundedPad1.0x1.5mm, F.Cu at (323.7, 155.0)
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Routing:
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