File: Gov_TrkU_panel/Gov_tracker_Panel/Gov_tracker_Panel.kicad_pcb (KiCad board)
At the start: 2 copper layers, 320 x 136 mm, 689 parts, among them CN1 Main_Connector, CN2 Main_Connector, CN3 Main_Connector, CN4 Main_Connector, J1 Conn_01x02, J10 Prog_T, J11 Debug, J12 USB_B_Mini, J13 USB_Con, J14 ANT, J15 Conn_Coaxial, J16 Debug/GPS_DBG, J17 Conn_Coaxial, J18 Prog_G, J19 Prog_T, J2 USB_B_Mini, J20 Debug, J21 Conn_01x02, J22 USB_B_Mini, J23 USB_Con, J24 ANT, J25 Conn_Coaxial, J26 Debug/GPS_DBG, J27 Conn_Coaxial, J28 Prog_G, J29 Prog_T, J3 USB_Con, J30 Debug, J31 Conn_01x02, J32 USB_B_Mini, J33 USB_Con, J34 ANT, J35 Conn_Coaxial, J36 Debug/GPS_DBG, J37 Conn_Coaxial, J38 Prog_G, J39 Prog_T, J4 ANT, J40 Debug, J5 Conn_Coaxial, J6 Debug/GPS_DBG, J7 Conn_Coaxial, J8 Conn_01x02, J9 Prog_G, K2 G5Q-1, K3 SRA-05VDC-CL, K4 G5Q-1, K5 SRA-05VDC-CL, K6 G5Q-1, K7 SRA-05VDC-CL, K8 G5Q-1, K9 SRA-05VDC-CL, Q1 SI2333DS, Q10 BC817, Q11 SI2333DS, Q12 BC817, Q13 BC817, Q14 BSS84, Q15 BC817, Q16 SI2333DS, Q17 BC817, Q18 BC817, Q19 BSS84, Q2 BC817, Q20 BC817, Q3 BC817, Q4 BSS84, Q5 BC817, Q6 SI2333DS, Q7 BC817, Q8 BC817, Q9 BSS84, U10 LM2596S-5, U11 LM393, U12 W25Q128JVS, U13 STM32F103RCTx, U14 NEO-6M-GPS, U15 SY7208B, U16 LM1117-3.3, U17 MCP73831-5-OT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

Commit message: 5.2.6 final edit
Parts:
- removed 3.3V1, 3.3V2, 3.3V3: 3.3V, TestPoint:TestPoint_Pad_1.0x1.0mm
- removed 5V1, 5V2, 5V3: 5V, TestPoint:TestPoint_Pad_1.0x1.0mm
- removed BT2, BT3, BT4: 1056, 1056:BAT_1056
- removed BZ2, BZ3, BZ4: Buzzer, Buzzer_Beeper:MagneticBuzzer_ProSignal_ABI-009-RC
- removed C100, C101, C146, C147, C54, C55: 10uF/25V, Capacitor_THT:CP_Radial_D5.0mm_P2.50mm
- removed C102, C148, C56: 1uF/16V, Capacitor_SMD:C_0603_1608Metric
- removed C103, C149, C57: 0.1uF/16V, Capacitor_SMD:C_0603_1608Metric
- removed C104, C150, C58: 100uFx6.3v, Capacitor_SMD:C_Elec_5x5.8
- removed C105, C151, C59: 220uF/10v, Capacitor_SMD:CP_Elec_8x6.5
- removed C106, C118, C152, C164, C60, C72: 0.1uFx/10V, Capacitor_SMD:C_0805_2012Metric
- removed C107, C138, C142, C143, C153, C184, C50, C51, C61, C92, C96, C97: 1uF, Capacitor_SMD:C_0603_1608Metric
- removed C108, C109, C132, C133, C154, C155, C178, C179, C62, C63, C86, C87: 18pF, Capacitor_SMD:C_0603_1608Metric
- removed C110, C112, C114, C116, C119, C121, C134, C136, C156, C158, C160, C162, C165, C167, C180, C182, C64, C66, C68, C70, C73, C75, C88, C90: 1uF/6.3V, Capacitor_SMD:C_0603_1608Metric
- removed C111, C113, C115, C117, C120, C122, C135, C137, C157, C159, C161, C163, C166, C168, C181, C183, C65, C67, C69, C71, C74, C76, C89, C91: 0.1uF/6.3V, Capacitor_SMD:C_0603_1608Metric
- removed C123, C124, C125, C126, C127, C169, C170, C171, C172, C173, C77, C78, C79, C80, C81: 0.1uF, Capacitor_SMD:C_0603_1608Metric
- removed C128, C131, C174, C177, C82, C85: 22pF, Capacitor_SMD:C_0603_1608Metric
- removed C129, C175, C83: 330uF, Capacitor_Tantalum_SMD:CP_EIA-6032-15_Kemet-U
- removed C130, C176, C84: 10uFx/10V, Capacitor_SMD:C_0603_1608Metric
- removed C139, C141, C3, C49, C93, C95: 220uF/25V, Capacitor_SMD:CP_Elec_8x6.9
- removed C140, C48, C94: 10uFx16v, Capacitor_SMD:C_0603_1608Metric
- removed C144, C145, C52, C53, C98, C99: 10uF/16V, Capacitor_SMD:C_0603_1608Metric
- removed CN2, CN3, CN4: Main_Connector, 66201821122:66201821122
- removed D24, D33, D34, D38, D44, D45, D47, D56, D57, D61, D67, D68, D70, D79, D80, D84, D90, D91: 3.9 Zener, Diode_SMD:D_SOD-123
- removed D25, D26, D28, D30, D48, D49, D51, D53, D71, D72, D74, D76: Schottkey/1A, Diode_SMD:D_SMA
- removed D27, D50, D73: R_LED, LED_SMD:LED_0805_2012Metric
- removed D29, D52, D75: G_LED, LED_SMD:LED_0805_2012Metric
- removed D31, D54, D77: GPRS_LED, LED_SMD:LED_0805_2012Metric
- removed D32, D43, D55, D66, D78, D89: G_Purpose, Diode_SMD:D_SMA
- removed D35, D58, D81: PW_LED, LED_SMD:LED_0805_2012Metric
- removed D36, D59, D82: Power, LED_SMD:LED_0805_2012Metric
- removed D37, D60, D83: Schottkey, Diode_SMD:D_SOD-123
- removed D39, D62, D85: G_purpose, Diode_SMD:D_SMA
- removed D40, D63, D86: ST, LED_SMD:LED_0805_2012Metric
- removed D41, D64, D87: NW, LED_SMD:LED_0805_2012Metric
- removed D42, D65, D88: 1N4148, Diode_SMD:D_SOD-123
- removed D46, D69, D92: ?, Diode_SMD:D_SMA
- removed F2, F3, F4: 30V/0.09A, Fuse:Fuse_BelFuse_0ZRE0005FF_L8.3mm_W3.8mm
- removed FID10, FID16, FID22: Fiducial, Fiducial:Fiducial_1.5mm_Mask3mm
- removed FID11, FID12, FID17, FID18, FID23, FID24: Fiducial, Fiducial:Fiducial_0.75mm_Mask1.5mm
- removed FID13, FID14, FID15, FID19, FID20, FID21, FID7, FID8, FID9: Fiducial, Fiducial:Fiducial_1mm_Mask3mm
- removed J12, J22, J32: USB_B_Mini, Connector_USB:USB_Mini-B_Lumberg_2486_01_Horizontal
- removed J13, J23, J33: USB_Con, Connector_PinSocket_2.54mm:PinSocket_1x04_P2.54mm_Vertical
- removed J14, J24, J34: ANT, Connector_Coaxial:SMA_Amphenol_132291_Vertical
- removed J15, J25, J35: Conn_Coaxial, Connector_Coaxial:SMA_Amphenol_132291_Vertical
- removed J16, J26, J36: Debug/GPS_DBG, Connector_PinSocket_2.54mm:PinSocket_1x05_P2.54mm_Vertical
- removed J17, J27, J37: Conn_Coaxial, Connector_Coaxial:U.FL_Molex_MCRF_73412-0110_Vertical
- removed J18, J28, J38: Prog_G, Connector_PinSocket_2.54mm:PinSocket_1x06_P2.54mm_Vertical
- removed J19, J29, J39: Prog_T, Connector_PinSocket_2.54mm:PinSocket_1x06_P2.54mm_Vertical
- removed J20, J30, J40: Debug, Connector_PinHeader_2.54mm:PinHeader_1x03_P2.54mm_Vertical
- removed J21, J31, J8: Conn_01x02, Connector_JST:JST_PH_B2B-PH-K_1x02_P2.00mm_Vertical
- removed JP2, JP3, JP4: Analog fuel jumper, Jumper:SolderJumper-2_P1.3mm_Open_RoundedPad1.0x1.5mm
- removed K4, K6, K8: G5Q-1, Relay_THT:Relay_SPDT_Omron-G5LE-1
- removed K5, K7, K9: SRA-05VDC-CL, SRA-05VDC-CL:RELAY_SRA-05VDC-CL
- removed L10, L3, L7: L-US, Inductor_SMD:L_Taiyo-Yuden_NR-60xx
- removed L11, L4, L8: INDUCTOR, Inductor_SMD:L_Pulse_PA4320
- removed L12, L6, L9: 22nH, Inductor_SMD:L_1206_3216Metric
- removed Q10, Q12, Q13, Q15, Q17, Q18, Q20, Q7, Q8: BC817, Package_TO_SOT_SMD:SOT-23
- removed Q11, Q16, Q6: SI2333DS, Package_TO_SOT_SMD:SC-59
- removed Q14, Q19, Q9: BSS84, Package_TO_SOT_SMD:SOT-23
- removed R100, R126, R145, R150, R176, R195, R200, R76, R95: 100k, Resistor_SMD:R_0603_1608Metric
- removed R101, R105, R106, R107, R114, R116, R121, R125, R127, R139, R148, R149, R151, R155, R156, R157, R164, R166, R171, R175, R177, R189, R198, R199, R201, R55, R56, R57, R64, R66, R71, R75, R77, R89, R98, R99: 1k, Resistor_SMD:R_0603_1608Metric
- removed R102, R152, R202: 22, Resistor_SMD:R_0603_1608Metric
- removed R103, R104, R111, R113, R120, R122, R123, R124, R128, R129, R130, R131, R133, R136, R143, R144, R146, R153, R154, R161, R163, R170, R172, R173, R174, R178, R179, R180, R181, R183, R186, R193, R194, R196, R46, R48, R61, R63, R70, R72, R73, R74, R78, R79, R80, R81, R83, R86, R93, R94, R96: 10k, Resistor_SMD:R_0603_1608Metric
- removed R108, R158, R58: 8.2k, Resistor_SMD:R_0603_1608Metric
- removed R109, R159, R59: 1.1k, Resistor_SMD:R_0603_1608Metric
- removed R110, R112, R160, R162, R60, R62: 33k, Resistor_SMD:R_0603_1608Metric
- removed R115, R165, R65: 5.1k, Resistor_SMD:R_0603_1608Metric
- removed R117, R167, R67: 2k, Resistor_SMD:R_0603_1608Metric
- removed R118, R119, R168, R169, R68, R69: 33, Resistor_SMD:R_0603_1608Metric
- removed R132, R137, R138, R140, R141, R142, R182, R187, R188, R190, R191, R192, R82, R87, R88, R90, R91, R92: 10K, Resistor_SMD:R_0603_1608Metric
- removed R134, R135, R184, R185, R84, R85: 1K(1%)0.1W, Resistor_SMD:R_0603_1608Metric
- removed R147, R197, R97: 3.3k, Resistor_SMD:R_0603_1608Metric
- removed TP5, TP6, TP7: BT, TestPoint:TestPoint_Pad_1.0x1.0mm
- removed U10, U26, U38: LM2596S-5, Package_TO_SOT_SMD:TO-263-5_TabPin3
- removed U15, U27, U39: SY7208B, Package_TO_SOT_SMD:SOT-23-6
- removed U16, U28, U40: LM1117-3.3, Package_TO_SOT_SMD:SOT-223-3_TabPin2
- removed U17, U29, U41: MCP73831-5-OT, Package_TO_SOT_SMD:SOT-23-5
- removed U18, U24, U30, U36, U42, U48: STM32F103RCTx, Package_QFP:LQFP-64_10x10mm_P0.5mm
- removed U19, U31, U43: 693021020811, simcard:693021020811
- removed U20, U32, U44: SIM800C, RF_GSM:SIMCom_SIM800C
- removed U21, U33, U45: MAX3232, MAX3232EUE:SOP65P640X110-16N
- removed U22, U34, U46: LM393, LM393:SO08
- removed U23, U35, U47: W25Q128JVS, Package_SO:SOIC-8_5.23x5.23mm_P1.27mm
- removed U25, U37, U49: NEO-6M-GPS, NEO-6M-GPS:XCVR_NEO-6M-GPS
- removed Y10, Y12, Y2, Y3, Y7, Y9: 8MHz, Crystal:Crystal_HC49-U_Vertical
- removed Y11, Y6, Y8: 32.678kHz, Crystal:Crystal_DS10_D1.0mm_L4.3mm_Vertical
- added 3.3V: 3.3V, TestPoint:TestPoint_Pad_1.0x1.0mm, F.Cu at (304.9, 128.7)
- added 3.3V: 3.3V, TestPoint:TestPoint_Pad_1.0x1.0mm, F.Cu at (229.9, 128.7)
- added 3.3V: 3.3V, TestPoint:TestPoint_Pad_1.0x1.0mm, F.Cu at (154.9, 128.7)
- added 5V: 5V, TestPoint:TestPoint_Pad_1.0x1.0mm, F.Cu at (154.2, 119.8)
- added 5V: 5V, TestPoint:TestPoint_Pad_1.0x1.0mm, F.Cu at (304.2, 119.8)
- added 5V: 5V, TestPoint:TestPoint_Pad_1.0x1.0mm, F.Cu at (229.2, 119.8)
- added BT1: 1056, 1056:BAT_1056, B.Cu at (187.3, 124.5)
- added BT1: 1056, 1056:BAT_1056, B.Cu at (262.3, 124.5)
- added BT1: 1056, 1056:BAT_1056, B.Cu at (337.3, 124.5)
- added BZ1: Buzzer, Buzzer_Beeper:MagneticBuzzer_ProSignal_ABI-009-RC, F.Cu at (266.4, 122.8)
- added BZ1: Buzzer, Buzzer_Beeper:MagneticBuzzer_ProSignal_ABI-009-RC, F.Cu at (341.4, 122.8)
- added BZ1: Buzzer, Buzzer_Beeper:MagneticBuzzer_ProSignal_ABI-009-RC, F.Cu at (191.4, 122.8)
- added C1: 220uF/25V, Capacitor_SMD:CP_Elec_8x6.9, F.Cu at (313.7, 163.1)
- added C1: 220uF/25V, Capacitor_SMD:CP_Elec_8x6.9, F.Cu at (238.7, 163.1)
- added C1: 220uF/25V, Capacitor_SMD:CP_Elec_8x6.9, F.Cu at (163.7, 163.1)
- added C10: 10uF/25V, Capacitor_THT:CP_Radial_D5.0mm_P2.50mm, F.Cu at (154.8, 136.0)
- added C10: 10uF/25V, Capacitor_THT:CP_Radial_D5.0mm_P2.50mm, F.Cu at (304.8, 136.0)
- added C10: 10uF/25V, Capacitor_THT:CP_Radial_D5.0mm_P2.50mm, F.Cu at (229.8, 136.0)
- added C11: 1uF/16V, Capacitor_SMD:C_0603_1608Metric, B.Cu at (230.5, 139.2)
- added C11: 1uF/16V, Capacitor_SMD:C_0603_1608Metric, B.Cu at (305.5, 139.2)
- added C11: 1uF/16V, Capacitor_SMD:C_0603_1608Metric, B.Cu at (155.5, 139.2)
- added C12: 0.1uF/16V, Capacitor_SMD:C_0603_1608Metric, F.Cu at (357.6, 151.8)
- added C12: 0.1uF/16V, Capacitor_SMD:C_0603_1608Metric, F.Cu at (207.6, 151.8)
- added C12: 0.1uF/16V, Capacitor_SMD:C_0603_1608Metric, F.Cu at (282.6, 151.8)
- added C13: 100uFx6.3v, Capacitor_SMD:C_Elec_5x5.8, F.Cu at (249.0, 183.0)
- added C13: 100uFx6.3v, Capacitor_SMD:C_Elec_5x5.8, F.Cu at (174.0, 183.0)
- added C13: 100uFx6.3v, Capacitor_SMD:C_Elec_5x5.8, F.Cu at (324.0, 183.0)
- added C14: 220uF/10v, Capacitor_SMD:CP_Elec_8x6.5, F.Cu at (247.4, 174.2)
- added C14: 220uF/10v, Capacitor_SMD:CP_Elec_8x6.5, F.Cu at (172.4, 174.2)
- added C14: 220uF/10v, Capacitor_SMD:CP_Elec_8x6.5, F.Cu at (322.4, 174.2)
- added C15: 0.1uFx/10V, Capacitor_SMD:C_0805_2012Metric, F.Cu at (323.0, 165.4)
- added C15: 0.1uFx/10V, Capacitor_SMD:C_0805_2012Metric, F.Cu at (248.0, 165.4)
- added C15: 0.1uFx/10V, Capacitor_SMD:C_0805_2012Metric, F.Cu at (173.0, 165.4)
- added C16: 1uF, Capacitor_SMD:C_0603_1608Metric, F.Cu at (336.9, 144.2)
- added C16: 1uF, Capacitor_SMD:C_0603_1608Metric, F.Cu at (186.9, 144.2)
- added C16: 1uF, Capacitor_SMD:C_0603_1608Metric, F.Cu at (261.9, 144.2)
- added C17: 18pF, Capacitor_SMD:C_0603_1608Metric, F.Cu at (193.0, 141.5)
- added C17: 18pF, Capacitor_SMD:C_0603_1608Metric, F.Cu at (343.0, 141.5)
- added C17: 18pF, Capacitor_SMD:C_0603_1608Metric, F.Cu at (268.0, 141.5)
- added C18: 18pF, Capacitor_SMD:C_0603_1608Metric, F.Cu at (346.8, 141.6)
- added C18: 18pF, Capacitor_SMD:C_0603_1608Metric, F.Cu at (196.8, 141.6)
- added C18: 18pF, Capacitor_SMD:C_0603_1608Metric, F.Cu at (271.8, 141.6)
- added C19: 1uF/6.3V, Capacitor_SMD:C_0603_1608Metric, F.Cu at (178.9, 119.9)
- added C19: 1uF/6.3V, Capacitor_SMD:C_0603_1608Metric, F.Cu at (328.9, 119.9)
- added C19: 1uF/6.3V, Capacitor_SMD:C_0603_1608Metric, F.Cu at (253.9, 119.9)
- added C2: 10uFx16v, Capacitor_SMD:C_0603_1608Metric, B.Cu at (205.5, 164.3)
- added C2: 10uFx16v, Capacitor_SMD:C_0603_1608Metric, B.Cu at (355.5, 164.3)
- added C2: 10uFx16v, Capacitor_SMD:C_0603_1608Metric, B.Cu at (280.5, 164.3)
- added C20: 0.1uF/6.3V, Capacitor_SMD:C_0603_1608Metric, F.Cu at (328.9, 121.7)
- added C20: 0.1uF/6.3V, Capacitor_SMD:C_0603_1608Metric, F.Cu at (253.9, 121.7)
- added C20: 0.1uF/6.3V, Capacitor_SMD:C_0603_1608Metric, F.Cu at (178.9, 121.7)
- added C21: 1uF/6.3V, Capacitor_SMD:C_0603_1608Metric, F.Cu at (169.9, 121.6)
- added C21: 1uF/6.3V, Capacitor_SMD:C_0603_1608Metric, F.Cu at (319.9, 121.6)
- added C21: 1uF/6.3V, Capacitor_SMD:C_0603_1608Metric, F.Cu at (244.9, 121.6)
- added C22: 0.1uF/6.3V, Capacitor_SMD:C_0603_1608Metric, F.Cu at (319.8, 119.7)
- added C22: 0.1uF/6.3V, Capacitor_SMD:C_0603_1608Metric, F.Cu at (244.8, 119.7)
- added C22: 0.1uF/6.3V, Capacitor_SMD:C_0603_1608Metric, F.Cu at (169.8, 119.7)
- added C23: 1uF/6.3V, Capacitor_SMD:C_0603_1608Metric, F.Cu at (239.1, 140.5)
- added C23: 1uF/6.3V, Capacitor_SMD:C_0603_1608Metric, F.Cu at (314.1, 140.5)
- added C23: 1uF/6.3V, Capacitor_SMD:C_0603_1608Metric, F.Cu at (164.1, 140.5)
- added C24: 0.1uF/6.3V, Capacitor_SMD:C_0603_1608Metric, F.Cu at (313.3, 136.6)
- added C24: 0.1uF/6.3V, Capacitor_SMD:C_0603_1608Metric, F.Cu at (238.3, 136.6)
- added C24: 0.1uF/6.3V, Capacitor_SMD:C_0603_1608Metric, F.Cu at (163.3, 136.6)
- added C25: 1uF/6.3V, Capacitor_SMD:C_0603_1608Metric, F.Cu at (332.7, 135.6)
- added C25: 1uF/6.3V, Capacitor_SMD:C_0603_1608Metric, F.Cu at (257.7, 135.6)
- added C25: 1uF/6.3V, Capacitor_SMD:C_0603_1608Metric, F.Cu at (182.7, 135.6)
- added C26: 0.1uF/6.3V, Capacitor_SMD:C_0603_1608Metric, F.Cu at (184.6, 135.7)
- added C26: 0.1uF/6.3V, Capacitor_SMD:C_0603_1608Metric, F.Cu at (259.6, 135.7)
- added C26: 0.1uF/6.3V, Capacitor_SMD:C_0603_1608Metric, F.Cu at (334.6, 135.7)
- added C27: 0.1uFx/10V, Capacitor_SMD:C_0805_2012Metric, F.Cu at (328.5, 168.0)
- added C27: 0.1uFx/10V, Capacitor_SMD:C_0805_2012Metric, F.Cu at (178.5, 168.0)
- added C27: 0.1uFx/10V, Capacitor_SMD:C_0805_2012Metric, F.Cu at (253.5, 168.0)
- added C28: 1uF/6.3V, Capacitor_SMD:C_0603_1608Metric, F.Cu at (187.1, 131.6)
- added C28: 1uF/6.3V, Capacitor_SMD:C_0603_1608Metric, F.Cu at (337.1, 131.6)
- added C28: 1uF/6.3V, Capacitor_SMD:C_0603_1608Metric, F.Cu at (262.1, 131.6)
- added C29: 0.1uF/6.3V, Capacitor_SMD:C_0603_1608Metric, F.Cu at (188.7, 131.6)
- added C29: 0.1uF/6.3V, Capacitor_SMD:C_0603_1608Metric, F.Cu at (263.7, 131.6)
- added C29: 0.1uF/6.3V, Capacitor_SMD:C_0603_1608Metric, F.Cu at (338.7, 131.6)
- added C30: 1uF/6.3V, Capacitor_SMD:C_0603_1608Metric, F.Cu at (207.8, 129.3)
- added C30: 1uF/6.3V, Capacitor_SMD:C_0603_1608Metric, F.Cu at (357.8, 129.3)
- added C30: 1uF/6.3V, Capacitor_SMD:C_0603_1608Metric, F.Cu at (282.8, 129.3)
- added C31: 0.1uF/6.3V, Capacitor_SMD:C_0603_1608Metric, F.Cu at (284.9, 129.3)
- added C31: 0.1uF/6.3V, Capacitor_SMD:C_0603_1608Metric, F.Cu at (209.9, 129.3)
- added C31: 0.1uF/6.3V, Capacitor_SMD:C_0603_1608Metric, F.Cu at (359.9, 129.3)
- added C32: 0.1uF, Capacitor_SMD:C_0603_1608Metric, B.Cu at (313.5, 157.1)
- added C32: 0.1uF, Capacitor_SMD:C_0603_1608Metric, B.Cu at (163.5, 157.1)
- added C32: 0.1uF, Capacitor_SMD:C_0603_1608Metric, B.Cu at (238.5, 157.1)
- added C33: 0.1uF, Capacitor_SMD:C_0603_1608Metric, B.Cu at (323.3, 165.8)
- added C33: 0.1uF, Capacitor_SMD:C_0603_1608Metric, B.Cu at (248.3, 165.8)
- added C33: 0.1uF, Capacitor_SMD:C_0603_1608Metric, B.Cu at (173.3, 165.8)
- added C34: 0.1uF, Capacitor_SMD:C_0603_1608Metric, B.Cu at (245.6, 166.7)
- added C34: 0.1uF, Capacitor_SMD:C_0603_1608Metric, B.Cu at (320.6, 166.7)
- added C34: 0.1uF, Capacitor_SMD:C_0603_1608Metric, B.Cu at (170.6, 166.7)
- added C35: 0.1uF, Capacitor_SMD:C_0603_1608Metric, B.Cu at (317.0, 157.1)
- added C35: 0.1uF, Capacitor_SMD:C_0603_1608Metric, B.Cu at (167.0, 157.1)
- added C35: 0.1uF, Capacitor_SMD:C_0603_1608Metric, B.Cu at (242.0, 157.1)
- added C36: 0.1uF, Capacitor_SMD:C_0603_1608Metric, B.Cu at (317.0, 155.2)
- added C36: 0.1uF, Capacitor_SMD:C_0603_1608Metric, B.Cu at (167.0, 155.2)
- added C36: 0.1uF, Capacitor_SMD:C_0603_1608Metric, B.Cu at (242.0, 155.2)
- added C37: 22pF, Capacitor_SMD:C_0603_1608Metric, F.Cu at (245.3, 140.3)
- added C37: 22pF, Capacitor_SMD:C_0603_1608Metric, F.Cu at (320.3, 140.3)
- added C37: 22pF, Capacitor_SMD:C_0603_1608Metric, F.Cu at (170.3, 140.3)
- added C38: 330uF, Capacitor_Tantalum_SMD:CP_EIA-6032-15_Kemet-U, F.Cu at (179.0, 173.2)
- added C38: 330uF, Capacitor_Tantalum_SMD:CP_EIA-6032-15_Kemet-U, F.Cu at (254.0, 173.2)
- added C38: 330uF, Capacitor_Tantalum_SMD:CP_EIA-6032-15_Kemet-U, F.Cu at (329.0, 173.2)
- added C39: 10uFx/10V, Capacitor_SMD:C_0603_1608Metric, F.Cu at (253.6, 165.1)
- added C39: 10uFx/10V, Capacitor_SMD:C_0603_1608Metric, F.Cu at (178.6, 165.1)
- added C39: 10uFx/10V, Capacitor_SMD:C_0603_1608Metric, F.Cu at (328.6, 165.1)
- added C4: 220uF/25V, Capacitor_SMD:CP_Elec_8x6.9, F.Cu at (147.9, 143.6)
- added C4: 220uF/25V, Capacitor_SMD:CP_Elec_8x6.9, F.Cu at (297.9, 143.6)
- added C4: 220uF/25V, Capacitor_SMD:CP_Elec_8x6.9, F.Cu at (222.9, 143.6)
- added C40: 22pF, Capacitor_SMD:C_0603_1608Metric, F.Cu at (317.2, 140.3)
- added C40: 22pF, Capacitor_SMD:C_0603_1608Metric, F.Cu at (242.2, 140.3)
- added C40: 22pF, Capacitor_SMD:C_0603_1608Metric, F.Cu at (167.2, 140.3)
- added C41: 18pF, Capacitor_SMD:C_0603_1608Metric, F.Cu at (173.4, 140.3)
- added C41: 18pF, Capacitor_SMD:C_0603_1608Metric, F.Cu at (248.4, 140.3)
- added C41: 18pF, Capacitor_SMD:C_0603_1608Metric, F.Cu at (323.4, 140.3)
- added C42: 18pF, Capacitor_SMD:C_0603_1608Metric, F.Cu at (251.5, 140.3)
- added C42: 18pF, Capacitor_SMD:C_0603_1608Metric, F.Cu at (176.5, 140.3)
- added C42: 18pF, Capacitor_SMD:C_0603_1608Metric, F.Cu at (326.5, 140.3)
- added C43: 1uF/6.3V, Capacitor_SMD:C_0603_1608Metric, F.Cu at (279.1, 147.2)
- added C43: 1uF/6.3V, Capacitor_SMD:C_0603_1608Metric, F.Cu at (204.2, 147.2)
- added C43: 1uF/6.3V, Capacitor_SMD:C_0603_1608Metric, F.Cu at (354.1, 147.2)
- added C44: 0.1uF/6.3V, Capacitor_SMD:C_0603_1608Metric, F.Cu at (206.8, 147.2)
- added C44: 0.1uF/6.3V, Capacitor_SMD:C_0603_1608Metric, F.Cu at (281.8, 147.2)
- added C44: 0.1uF/6.3V, Capacitor_SMD:C_0603_1608Metric, F.Cu at (356.8, 147.2)
- added C45: 1uF/6.3V, Capacitor_SMD:C_0603_1608Metric, F.Cu at (187.9, 135.8)
- added C45: 1uF/6.3V, Capacitor_SMD:C_0603_1608Metric, F.Cu at (337.9, 135.8)
- added C45: 1uF/6.3V, Capacitor_SMD:C_0603_1608Metric, F.Cu at (262.9, 135.8)
- added C46: 0.1uF/6.3V, Capacitor_SMD:C_0603_1608Metric, F.Cu at (337.9, 137.7)
- added C46: 0.1uF/6.3V, Capacitor_SMD:C_0603_1608Metric, F.Cu at (187.9, 137.7)
- added C46: 0.1uF/6.3V, Capacitor_SMD:C_0603_1608Metric, F.Cu at (262.9, 137.7)
- added C47: 1uF, Capacitor_SMD:C_0603_1608Metric, B.Cu at (173.1, 162.3)
- added C47: 1uF, Capacitor_SMD:C_0603_1608Metric, B.Cu at (323.1, 162.3)
- added C47: 1uF, Capacitor_SMD:C_0603_1608Metric, B.Cu at (248.1, 162.3)
- added C5: 1uF, Capacitor_SMD:C_0603_1608Metric, B.Cu at (237.3, 139.3)
- added C5: 1uF, Capacitor_SMD:C_0603_1608Metric, B.Cu at (162.3, 139.3)
- added C5: 1uF, Capacitor_SMD:C_0603_1608Metric, B.Cu at (312.3, 139.3)
- added C6: 1uF, Capacitor_SMD:C_0603_1608Metric, F.Cu at (232.0, 149.0)
- added C6: 1uF, Capacitor_SMD:C_0603_1608Metric, F.Cu at (307.0, 149.0)
- added C6: 1uF, Capacitor_SMD:C_0603_1608Metric, F.Cu at (157.0, 149.0)
- added C7: 10uF/16V, Capacitor_SMD:C_0603_1608Metric, F.Cu at (209.3, 159.4)
- added C7: 10uF/16V, Capacitor_SMD:C_0603_1608Metric, F.Cu at (284.3, 159.4)
- added C7: 10uF/16V, Capacitor_SMD:C_0603_1608Metric, F.Cu at (359.3, 159.4)
- added C8: 10uF/16V, Capacitor_SMD:C_0603_1608Metric, F.Cu at (285.0, 163.0)
- added C8: 10uF/16V, Capacitor_SMD:C_0603_1608Metric, F.Cu at (360.0, 163.0)
- added C8: 10uF/16V, Capacitor_SMD:C_0603_1608Metric, F.Cu at (210.0, 163.0)
- added C9: 10uF/25V, Capacitor_THT:CP_Radial_D5.0mm_P2.50mm, F.Cu at (306.7, 142.0)
- added C9: 10uF/25V, Capacitor_THT:CP_Radial_D5.0mm_P2.50mm, F.Cu at (156.7, 142.0)
- added C9: 10uF/25V, Capacitor_THT:CP_Radial_D5.0mm_P2.50mm, F.Cu at (231.7, 142.0)
- added CN1: Main_Connector, 66201821122:66201821122, F.Cu at (317.9, 190.6)
- added CN1: Main_Connector, 66201821122:66201821122, F.Cu at (167.9, 190.6)
- added CN1: Main_Connector, 66201821122:66201821122, F.Cu at (242.9, 190.6)
- added D1: 3.9 Zener, Diode_SMD:D_SOD-123, F.Cu at (314.7, 178.4)
- added D1: 3.9 Zener, Diode_SMD:D_SOD-123, F.Cu at (239.7, 178.4)
- added D1: 3.9 Zener, Diode_SMD:D_SOD-123, F.Cu at (164.7, 178.4)
- added D10: 3.9 Zener, Diode_SMD:D_SOD-123, B.Cu at (273.0, 131.5)
- added D10: 3.9 Zener, Diode_SMD:D_SOD-123, B.Cu at (348.0, 131.5)
- added D10: 3.9 Zener, Diode_SMD:D_SOD-123, B.Cu at (198.0, 131.5)
- added D11: 3.9 Zener, Diode_SMD:D_SOD-123, B.Cu at (279.1, 128.3)
- added D11: 3.9 Zener, Diode_SMD:D_SOD-123, B.Cu at (204.1, 128.3)
- added D11: 3.9 Zener, Diode_SMD:D_SOD-123, B.Cu at (354.1, 128.3)
- added D12: PW_LED, LED_SMD:LED_0805_2012Metric, F.Cu at (220.1, 128.3)
- added D12: PW_LED, LED_SMD:LED_0805_2012Metric, F.Cu at (295.1, 128.3)
- added D12: PW_LED, LED_SMD:LED_0805_2012Metric, F.Cu at (145.1, 128.3)
- added D13: Power, LED_SMD:LED_0805_2012Metric, F.Cu at (271.9, 156.2)
- added D13: Power, LED_SMD:LED_0805_2012Metric, F.Cu at (346.9, 156.2)
- added D13: Power, LED_SMD:LED_0805_2012Metric, F.Cu at (196.9, 156.2)
- added D14: Schottkey, Diode_SMD:D_SOD-123, B.Cu at (284.1, 179.6)
- added D14: Schottkey, Diode_SMD:D_SOD-123, B.Cu at (209.1, 179.6)
- added D14: Schottkey, Diode_SMD:D_SOD-123, B.Cu at (359.1, 179.6)
- added D15: 3.9 Zener, Diode_SMD:D_SOD-123, F.Cu at (165.8, 121.2)
- added D15: 3.9 Zener, Diode_SMD:D_SOD-123, F.Cu at (240.8, 121.2)
- added D15: 3.9 Zener, Diode_SMD:D_SOD-123, F.Cu at (315.8, 121.2)
- added D16: G_purpose, Diode_SMD:D_SMA, B.Cu at (328.4, 162.7)
- added D16: G_purpose, Diode_SMD:D_SMA, B.Cu at (253.4, 162.7)
- added D16: G_purpose, Diode_SMD:D_SMA, B.Cu at (178.4, 162.7)
- added D17: ST, LED_SMD:LED_0805_2012Metric, F.Cu at (208.8, 173.3)
- added D17: ST, LED_SMD:LED_0805_2012Metric, F.Cu at (283.8, 173.3)
- added D17: ST, LED_SMD:LED_0805_2012Metric, F.Cu at (358.8, 173.3)
- added D18: NW, LED_SMD:LED_0805_2012Metric, F.Cu at (283.7, 170.3)
- added D18: NW, LED_SMD:LED_0805_2012Metric, F.Cu at (358.7, 170.3)
- added D18: NW, LED_SMD:LED_0805_2012Metric, F.Cu at (208.7, 170.3)
- added D19: 1N4148, Diode_SMD:D_SOD-123, F.Cu at (161.9, 139.9)
- added D19: 1N4148, Diode_SMD:D_SOD-123, F.Cu at (311.9, 139.9)
- added D19: 1N4148, Diode_SMD:D_SOD-123, F.Cu at (236.9, 139.9)
- added D2: Schottkey/1A, Diode_SMD:D_SMA, B.Cu at (225.3, 162.5)
- added D2: Schottkey/1A, Diode_SMD:D_SMA, B.Cu at (150.3, 162.5)
- added D2: Schottkey/1A, Diode_SMD:D_SMA, B.Cu at (300.3, 162.5)
- added D20: G_Purpose, Diode_SMD:D_SMA, B.Cu at (166.4, 182.3)
- added D20: G_Purpose, Diode_SMD:D_SMA, B.Cu at (241.4, 182.3)
- added D20: G_Purpose, Diode_SMD:D_SMA, B.Cu at (316.4, 182.3)
- added D21: 3.9 Zener, Diode_SMD:D_SOD-123, B.Cu at (180.4, 150.0)
- added D21: 3.9 Zener, Diode_SMD:D_SOD-123, B.Cu at (330.4, 150.0)
- added D21: 3.9 Zener, Diode_SMD:D_SOD-123, B.Cu at (255.4, 150.0)
- added D22: 3.9 Zener, Diode_SMD:D_SOD-123, F.Cu at (248.0, 160.4)
- added D22: 3.9 Zener, Diode_SMD:D_SOD-123, F.Cu at (323.0, 160.4)
- added D22: 3.9 Zener, Diode_SMD:D_SOD-123, F.Cu at (173.0, 160.4)
- added D23: ?, Diode_SMD:D_SMA, B.Cu at (159.9, 172.8)
- added D23: ?, Diode_SMD:D_SMA, B.Cu at (309.9, 172.8)
- added D23: ?, Diode_SMD:D_SMA, B.Cu at (234.9, 172.8)
- added D3: Schottkey/1A, Diode_SMD:D_SMA, B.Cu at (294.4, 155.2)
- added D3: Schottkey/1A, Diode_SMD:D_SMA, B.Cu at (219.3, 155.2)
- added D3: Schottkey/1A, Diode_SMD:D_SMA, B.Cu at (144.3, 155.2)
- added D4: R_LED, LED_SMD:LED_0805_2012Metric, F.Cu at (219.3, 123.9)
- added D4: R_LED, LED_SMD:LED_0805_2012Metric, F.Cu at (144.3, 123.9)
- added D4: R_LED, LED_SMD:LED_0805_2012Metric, F.Cu at (294.3, 123.9)
- added D5: Schottkey/1A, Diode_SMD:D_SMA, F.Cu at (164.4, 171.7)
- added D5: Schottkey/1A, Diode_SMD:D_SMA, F.Cu at (314.4, 171.7)
- added D5: Schottkey/1A, Diode_SMD:D_SMA, F.Cu at (239.4, 171.7)
- added D6: G_LED, LED_SMD:LED_0805_2012Metric, F.Cu at (147.0, 124.1)
- added D6: G_LED, LED_SMD:LED_0805_2012Metric, F.Cu at (222.0, 124.1)
- added D6: G_LED, LED_SMD:LED_0805_2012Metric, F.Cu at (297.0, 124.1)
- added D7: Schottkey/1A, Diode_SMD:D_SMA, B.Cu at (209.1, 169.2)
- added D7: Schottkey/1A, Diode_SMD:D_SMA, B.Cu at (284.1, 169.2)
- added D7: Schottkey/1A, Diode_SMD:D_SMA, B.Cu at (359.1, 169.2)
- added D8: GPRS_LED, LED_SMD:LED_0805_2012Metric, F.Cu at (225.1, 124.2)
- added D8: GPRS_LED, LED_SMD:LED_0805_2012Metric, F.Cu at (300.1, 124.2)
- added D8: GPRS_LED, LED_SMD:LED_0805_2012Metric, F.Cu at (150.1, 124.2)
- added D9: G_Purpose, Diode_SMD:D_SMA, B.Cu at (221.7, 148.5)
- added D9: G_Purpose, Diode_SMD:D_SMA, B.Cu at (146.7, 148.5)
- added D9: G_Purpose, Diode_SMD:D_SMA, B.Cu at (296.7, 148.5)
- added F1: 30V/0.09A, Fuse:Fuse_BelFuse_0ZRE0005FF_L8.3mm_W3.8mm, F.Cu at (309.5, 184.5)
- added F1: 30V/0.09A, Fuse:Fuse_BelFuse_0ZRE0005FF_L8.3mm_W3.8mm, F.Cu at (234.5, 184.5)
- added F1: 30V/0.09A, Fuse:Fuse_BelFuse_0ZRE0005FF_L8.3mm_W3.8mm, F.Cu at (159.5, 184.5)
- added FID1: Fiducial, Fiducial:Fiducial_1mm_Mask3mm, F.Cu at (291.0, 108.5)
- added FID1: Fiducial, Fiducial:Fiducial_1mm_Mask3mm, F.Cu at (141.0, 108.5)
- added FID1: Fiducial, Fiducial:Fiducial_1mm_Mask3mm, F.Cu at (216.0, 108.5)
- added FID2: Fiducial, Fiducial:Fiducial_1mm_Mask3mm, F.Cu at (216.0, 194.5)
- added FID2: Fiducial, Fiducial:Fiducial_1mm_Mask3mm, F.Cu at (291.0, 194.5)
- added FID2: Fiducial, Fiducial:Fiducial_1mm_Mask3mm, F.Cu at (141.0, 194.5)
- added FID3: Fiducial, Fiducial:Fiducial_1mm_Mask3mm, F.Cu at (287.0, 108.5)
- added FID3: Fiducial, Fiducial:Fiducial_1mm_Mask3mm, F.Cu at (212.0, 108.5)
- added FID3: Fiducial, Fiducial:Fiducial_1mm_Mask3mm, F.Cu at (362.0, 108.5)
- added FID4: Fiducial, Fiducial:Fiducial_1.5mm_Mask3mm, B.Cu at (362.0, 108.5)
- added FID4: Fiducial, Fiducial:Fiducial_1.5mm_Mask3mm, B.Cu at (287.0, 108.5)
- added FID4: Fiducial, Fiducial:Fiducial_1.5mm_Mask3mm, B.Cu at (212.0, 108.5)
- added FID5: Fiducial, Fiducial:Fiducial_0.75mm_Mask1.5mm, B.Cu at (141.0, 194.5)
- added FID5: Fiducial, Fiducial:Fiducial_0.75mm_Mask1.5mm, B.Cu at (291.0, 194.5)
- added FID5: Fiducial, Fiducial:Fiducial_0.75mm_Mask1.5mm, B.Cu at (216.0, 194.5)
- added FID6: Fiducial, Fiducial:Fiducial_0.75mm_Mask1.5mm, B.Cu at (216.0, 108.5)
- added FID6: Fiducial, Fiducial:Fiducial_0.75mm_Mask1.5mm, B.Cu at (141.0, 108.5)
- added FID6: Fiducial, Fiducial:Fiducial_0.75mm_Mask1.5mm, B.Cu at (291.0, 108.5)
- added J1: Conn_01x02, Connector_JST:JST_PH_B2B-PH-K_1x02_P2.00mm_Vertical, B.Cu at (179.4, 153.6)
- added J1: Conn_01x02, Connector_JST:JST_PH_B2B-PH-K_1x02_P2.00mm_Vertical, B.Cu at (254.4, 153.6)
- added J1: Conn_01x02, Connector_JST:JST_PH_B2B-PH-K_1x02_P2.00mm_Vertical, B.Cu at (329.4, 153.6)
- added J10: Prog_T, Connector_PinSocket_2.54mm:PinSocket_1x06_P2.54mm_Vertical, F.Cu at (359.9, 115.5)
- added J10: Prog_T, Connector_PinSocket_2.54mm:PinSocket_1x06_P2.54mm_Vertical, F.Cu at (284.9, 115.5)
- added J10: Prog_T, Connector_PinSocket_2.54mm:PinSocket_1x06_P2.54mm_Vertical, F.Cu at (209.9, 115.5)
- added J11: Debug, Connector_PinHeader_2.54mm:PinHeader_1x03_P2.54mm_Vertical, F.Cu at (323.4, 115.8)
- added J11: Debug, Connector_PinHeader_2.54mm:PinHeader_1x03_P2.54mm_Vertical, F.Cu at (248.3, 115.8)
- added J11: Debug, Connector_PinHeader_2.54mm:PinHeader_1x03_P2.54mm_Vertical, F.Cu at (173.3, 115.8)
- added J2: USB_B_Mini, Connector_USB:USB_Mini-B_Lumberg_2486_01_Horizontal, F.Cu at (282.6, 191.2)
- added J2: USB_B_Mini, Connector_USB:USB_Mini-B_Lumberg_2486_01_Horizontal, F.Cu at (357.6, 191.2)
- added J2: USB_B_Mini, Connector_USB:USB_Mini-B_Lumberg_2486_01_Horizontal, F.Cu at (207.6, 191.2)
- added J3: USB_Con, Connector_PinSocket_2.54mm:PinSocket_1x04_P2.54mm_Vertical, F.Cu at (353.4, 184.7)
- added J3: USB_Con, Connector_PinSocket_2.54mm:PinSocket_1x04_P2.54mm_Vertical, F.Cu at (278.4, 184.7)
- added J3: USB_Con, Connector_PinSocket_2.54mm:PinSocket_1x04_P2.54mm_Vertical, F.Cu at (203.3, 184.7)
- added J4: ANT, Connector_Coaxial:SMA_Amphenol_132291_Vertical, F.Cu at (338.0, 191.2)
- added J4: ANT, Connector_Coaxial:SMA_Amphenol_132291_Vertical, F.Cu at (188.0, 191.2)
- added J4: ANT, Connector_Coaxial:SMA_Amphenol_132291_Vertical, F.Cu at (263.0, 191.2)
- added J5: Conn_Coaxial, Connector_Coaxial:SMA_Amphenol_132291_Vertical, F.Cu at (272.2, 191.3)
- added J5: Conn_Coaxial, Connector_Coaxial:SMA_Amphenol_132291_Vertical, F.Cu at (197.2, 191.3)
- added J5: Conn_Coaxial, Connector_Coaxial:SMA_Amphenol_132291_Vertical, F.Cu at (347.2, 191.3)
- added J6: Debug/GPS_DBG, Connector_PinSocket_2.54mm:PinSocket_1x05_P2.54mm_Vertical, F.Cu at (359.8, 119.7)
- added J6: Debug/GPS_DBG, Connector_PinSocket_2.54mm:PinSocket_1x05_P2.54mm_Vertical, F.Cu at (209.8, 119.7)
- added J6: Debug/GPS_DBG, Connector_PinSocket_2.54mm:PinSocket_1x05_P2.54mm_Vertical, F.Cu at (284.8, 119.7)
- added J7: Conn_Coaxial, Connector_Coaxial:U.FL_Molex_MCRF_73412-0110_Vertical, F.Cu at (181.8, 182.5)
- added J7: Conn_Coaxial, Connector_Coaxial:U.FL_Molex_MCRF_73412-0110_Vertical, F.Cu at (331.8, 182.5)
- added J7: Conn_Coaxial, Connector_Coaxial:U.FL_Molex_MCRF_73412-0110_Vertical, F.Cu at (256.8, 182.5)
- added J9: Prog_G, Connector_PinSocket_2.54mm:PinSocket_1x06_P2.54mm_Vertical, F.Cu at (311.0, 118.6)
- added J9: Prog_G, Connector_PinSocket_2.54mm:PinSocket_1x06_P2.54mm_Vertical, F.Cu at (236.0, 118.6)
- added J9: Prog_G, Connector_PinSocket_2.54mm:PinSocket_1x06_P2.54mm_Vertical, F.Cu at (161.0, 118.6)
- added JP1: Analog fuel jumper, Jumper:SolderJumper-2_P1.3mm_Open_RoundedPad1.0x1.5mm, F.Cu at (323.7, 155.0)
- added JP1: Analog fuel jumper, Jumper:SolderJumper-2_P1.3mm_Open_RoundedPad1.0x1.5mm, F.Cu at (248.7, 155.0)
- added JP1: Analog fuel jumper, Jumper:SolderJumper-2_P1.3mm_Open_RoundedPad1.0x1.5mm, F.Cu at (173.7, 155.0)
- added K2: G5Q-1, Relay_THT:Relay_SPDT_Omron-G5LE-1, F.Cu at (223.8, 166.4)
- added K2: G5Q-1, Relay_THT:Relay_SPDT_Omron-G5LE-1, F.Cu at (148.8, 166.4)
- added K2: G5Q-1, Relay_THT:Relay_SPDT_Omron-G5LE-1, F.Cu at (298.8, 166.4)
- added K3: SRA-05VDC-CL, SRA-05VDC-CL:RELAY_SRA-05VDC-CL, F.Cu at (150.2, 178.3)
- added K3: SRA-05VDC-CL, SRA-05VDC-CL:RELAY_SRA-05VDC-CL, F.Cu at (300.1, 178.3)
- added K3: SRA-05VDC-CL, SRA-05VDC-CL:RELAY_SRA-05VDC-CL, F.Cu at (225.2, 178.3)
- added L1: L-US, Inductor_SMD:L_Taiyo-Yuden_NR-60xx, F.Cu at (353.1, 156.6)
- added L1: L-US, Inductor_SMD:L_Taiyo-Yuden_NR-60xx, F.Cu at (203.1, 156.6)
- added L1: L-US, Inductor_SMD:L_Taiyo-Yuden_NR-60xx, F.Cu at (278.1, 156.6)
- added L2: INDUCTOR, Inductor_SMD:L_Pulse_PA4320, F.Cu at (315.4, 151.2)
- added L2: INDUCTOR, Inductor_SMD:L_Pulse_PA4320, F.Cu at (165.4, 151.2)
- added L2: INDUCTOR, Inductor_SMD:L_Pulse_PA4320, F.Cu at (240.4, 151.2)
- added L5: 22nH, Inductor_SMD:L_1206_3216Metric, B.Cu at (273.8, 186.2)
- added L5: 22nH, Inductor_SMD:L_1206_3216Metric, B.Cu at (198.8, 186.2)
- added L5: 22nH, Inductor_SMD:L_1206_3216Metric, B.Cu at (348.8, 186.2)
- added Q1: SI2333DS, Package_TO_SOT_SMD:SC-59, F.Cu at (253.7, 160.6)
- added Q1: SI2333DS, Package_TO_SOT_SMD:SC-59, F.Cu at (328.7, 160.6)
- added Q1: SI2333DS, Package_TO_SOT_SMD:SC-59, F.Cu at (178.7, 160.6)
- added Q2: BC817, Package_TO_SOT_SMD:SOT-23, B.Cu at (346.8, 139.6)
- added Q2: BC817, Package_TO_SOT_SMD:SOT-23, B.Cu at (271.8, 139.6)
- added Q2: BC817, Package_TO_SOT_SMD:SOT-23, B.Cu at (196.8, 139.6)
- added Q3: BC817, Package_TO_SOT_SMD:SOT-23, F.Cu at (234.9, 173.6)
- added Q3: BC817, Package_TO_SOT_SMD:SOT-23, F.Cu at (309.9, 173.6)
- added Q3: BC817, Package_TO_SOT_SMD:SOT-23, F.Cu at (159.9, 173.6)
- added Q4: BSS84, Package_TO_SOT_SMD:SOT-23, F.Cu at (183.8, 158.2)
- added Q4: BSS84, Package_TO_SOT_SMD:SOT-23, F.Cu at (258.8, 158.2)
- added Q4: BSS84, Package_TO_SOT_SMD:SOT-23, F.Cu at (333.8, 158.2)
- added Q5: BC817, Package_TO_SOT_SMD:SOT-23, B.Cu at (332.9, 136.5)
- added Q5: BC817, Package_TO_SOT_SMD:SOT-23, B.Cu at (257.9, 136.5)
- added Q5: BC817, Package_TO_SOT_SMD:SOT-23, B.Cu at (182.9, 136.5)
- added R10: 33k, Resistor_SMD:R_0603_1608Metric, B.Cu at (347.1, 133.7)
- added R10: 33k, Resistor_SMD:R_0603_1608Metric, B.Cu at (272.1, 133.7)
- added R10: 33k, Resistor_SMD:R_0603_1608Metric, B.Cu at (197.2, 133.7)
- added R11: 10k, Resistor_SMD:R_0603_1608Metric, B.Cu at (272.2, 129.4)
- added R11: 10k, Resistor_SMD:R_0603_1608Metric, B.Cu at (197.2, 129.4)
- added R11: 10k, Resistor_SMD:R_0603_1608Metric, B.Cu at (347.2, 129.4)
- added R12: 33k, Resistor_SMD:R_0603_1608Metric, B.Cu at (350.4, 127.5)
- added R12: 33k, Resistor_SMD:R_0603_1608Metric, B.Cu at (200.4, 127.5)
- added R12: 33k, Resistor_SMD:R_0603_1608Metric, B.Cu at (275.4, 127.5)
- added R13: 10k, Resistor_SMD:R_0603_1608Metric, B.Cu at (202.2, 127.5)
- added R13: 10k, Resistor_SMD:R_0603_1608Metric, B.Cu at (352.1, 127.5)
- added R13: 10k, Resistor_SMD:R_0603_1608Metric, B.Cu at (277.1, 127.5)
- added R14: 1k, Resistor_SMD:R_0603_1608Metric, B.Cu at (295.0, 131.1)
- added R14: 1k, Resistor_SMD:R_0603_1608Metric, B.Cu at (145.0, 131.1)
- added R14: 1k, Resistor_SMD:R_0603_1608Metric, B.Cu at (220.0, 131.1)
- added R15: 5.1k, Resistor_SMD:R_0603_1608Metric, F.Cu at (192.6, 157.4)
- added R15: 5.1k, Resistor_SMD:R_0603_1608Metric, F.Cu at (342.6, 157.4)
- added R15: 5.1k, Resistor_SMD:R_0603_1608Metric, F.Cu at (267.6, 157.4)
- added R16: 1k, Resistor_SMD:R_0603_1608Metric, B.Cu at (347.1, 135.9)
- added R16: 1k, Resistor_SMD:R_0603_1608Metric, B.Cu at (272.1, 135.9)
- added R16: 1k, Resistor_SMD:R_0603_1608Metric, B.Cu at (197.2, 135.9)
- added R17: 2k, Resistor_SMD:R_0603_1608Metric, F.Cu at (262.3, 157.4)
- added R17: 2k, Resistor_SMD:R_0603_1608Metric, F.Cu at (337.3, 157.4)
- added R17: 2k, Resistor_SMD:R_0603_1608Metric, F.Cu at (187.3, 157.4)
- added R18: 33, Resistor_SMD:R_0603_1608Metric, B.Cu at (206.8, 180.5)
- added R18: 33, Resistor_SMD:R_0603_1608Metric, B.Cu at (281.8, 180.5)
- added R18: 33, Resistor_SMD:R_0603_1608Metric, B.Cu at (356.8, 180.5)
- added R19: 33, Resistor_SMD:R_0603_1608Metric, B.Cu at (280.2, 180.5)
- added R19: 33, Resistor_SMD:R_0603_1608Metric, B.Cu at (355.2, 180.5)
- added R19: 33, Resistor_SMD:R_0603_1608Metric, B.Cu at (205.2, 180.5)
- added R20: 10k, Resistor_SMD:R_0603_1608Metric, F.Cu at (248.1, 119.6)
- added R20: 10k, Resistor_SMD:R_0603_1608Metric, F.Cu at (173.1, 119.6)
- added R20: 10k, Resistor_SMD:R_0603_1608Metric, F.Cu at (323.1, 119.6)
- added R21: 1k, Resistor_SMD:R_0603_1608Metric, B.Cu at (206.8, 177.4)
- added R21: 1k, Resistor_SMD:R_0603_1608Metric, B.Cu at (281.8, 177.4)
- added R21: 1k, Resistor_SMD:R_0603_1608Metric, B.Cu at (356.8, 177.4)
- added R22: 10k, Resistor_SMD:R_0603_1608Metric, F.Cu at (347.4, 153.1)
- added R22: 10k, Resistor_SMD:R_0603_1608Metric, F.Cu at (272.4, 153.1)
- added R22: 10k, Resistor_SMD:R_0603_1608Metric, F.Cu at (197.4, 153.1)
- added R23: 10k, Resistor_SMD:R_0603_1608Metric, F.Cu at (279.0, 151.8)
- added R23: 10k, Resistor_SMD:R_0603_1608Metric, F.Cu at (354.0, 151.8)
- added R23: 10k, Resistor_SMD:R_0603_1608Metric, F.Cu at (204.0, 151.8)
- added R24: 10k, Resistor_SMD:R_0603_1608Metric, F.Cu at (323.2, 121.6)
- added R24: 10k, Resistor_SMD:R_0603_1608Metric, F.Cu at (248.2, 121.6)
- added R24: 10k, Resistor_SMD:R_0603_1608Metric, F.Cu at (173.2, 121.6)
- added R25: 1k, Resistor_SMD:R_0603_1608Metric, F.Cu at (273.3, 160.2)
- added R25: 1k, Resistor_SMD:R_0603_1608Metric, F.Cu at (348.3, 160.2)
- added R25: 1k, Resistor_SMD:R_0603_1608Metric, F.Cu at (198.3, 160.2)
- added R26: 100k, Resistor_SMD:R_0603_1608Metric, F.Cu at (344.4, 160.2)
- added R26: 100k, Resistor_SMD:R_0603_1608Metric, F.Cu at (269.4, 160.2)
- added R26: 100k, Resistor_SMD:R_0603_1608Metric, F.Cu at (194.4, 160.2)
- added R27: 1k, Resistor_SMD:R_0603_1608Metric, F.Cu at (206.4, 161.8)
- added R27: 1k, Resistor_SMD:R_0603_1608Metric, F.Cu at (281.4, 161.8)
- added R27: 1k, Resistor_SMD:R_0603_1608Metric, F.Cu at (356.4, 161.8)
- added R28: 10k, Resistor_SMD:R_0603_1608Metric, F.Cu at (180.5, 148.2)
- added R28: 10k, Resistor_SMD:R_0603_1608Metric, F.Cu at (255.5, 148.2)
- added R28: 10k, Resistor_SMD:R_0603_1608Metric, F.Cu at (330.5, 148.2)
- added R29: 10k, Resistor_SMD:R_0603_1608Metric, F.Cu at (180.4, 150.7)
- added R29: 10k, Resistor_SMD:R_0603_1608Metric, F.Cu at (330.4, 150.7)
- added R29: 10k, Resistor_SMD:R_0603_1608Metric, F.Cu at (255.4, 150.7)
- added R3: 10k, Resistor_SMD:R_0603_1608Metric, F.Cu at (314.6, 184.2)
- added R3: 10k, Resistor_SMD:R_0603_1608Metric, F.Cu at (164.7, 184.2)
- added R3: 10k, Resistor_SMD:R_0603_1608Metric, F.Cu at (239.7, 184.2)
- added R30: 10k, Resistor_SMD:R_0603_1608Metric, F.Cu at (337.9, 134.0)
- added R30: 10k, Resistor_SMD:R_0603_1608Metric, F.Cu at (262.9, 134.0)
- added R30: 10k, Resistor_SMD:R_0603_1608Metric, F.Cu at (187.9, 134.0)
- added R31: 10k, Resistor_SMD:R_0603_1608Metric, F.Cu at (276.7, 147.2)
- added R31: 10k, Resistor_SMD:R_0603_1608Metric, F.Cu at (201.7, 147.2)
- added R31: 10k, Resistor_SMD:R_0603_1608Metric, F.Cu at (351.7, 147.2)
- added R32: 10K, Resistor_SMD:R_0603_1608Metric, B.Cu at (356.8, 143.6)
- added R32: 10K, Resistor_SMD:R_0603_1608Metric, B.Cu at (281.8, 143.6)
- added R32: 10K, Resistor_SMD:R_0603_1608Metric, B.Cu at (206.8, 143.6)
- added R33: 10k, Resistor_SMD:R_0603_1608Metric, F.Cu at (182.8, 139.6)
- added R33: 10k, Resistor_SMD:R_0603_1608Metric, F.Cu at (257.8, 139.6)
- added R33: 10k, Resistor_SMD:R_0603_1608Metric, F.Cu at (332.8, 139.6)
- added R34: 1K(1%)0.1W, Resistor_SMD:R_0603_1608Metric, B.Cu at (205.6, 166.3)
- added R34: 1K(1%)0.1W, Resistor_SMD:R_0603_1608Metric, B.Cu at (280.6, 166.3)
- added R34: 1K(1%)0.1W, Resistor_SMD:R_0603_1608Metric, B.Cu at (355.6, 166.3)
- added R35: 1K(1%)0.1W, Resistor_SMD:R_0603_1608Metric, B.Cu at (205.6, 168.4)
- added R35: 1K(1%)0.1W, Resistor_SMD:R_0603_1608Metric, B.Cu at (355.6, 168.4)
- added R35: 1K(1%)0.1W, Resistor_SMD:R_0603_1608Metric, B.Cu at (280.6, 168.4)
- added R36: 10k, Resistor_SMD:R_0603_1608Metric, F.Cu at (238.3, 134.8)
- added R36: 10k, Resistor_SMD:R_0603_1608Metric, F.Cu at (163.3, 134.8)
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Connections:
- 3.3V pad 1: (no net) -> +3V3
- 5V pad 1: (no net) -> +5V
- BT1 pad N: (no net) -> GND
- BT1 pad P: (no net) -> BAT1
- BZ1 pad 1: (no net) -> +5V
- BZ1 pad 2: (no net) -> Net-(BZ1-+)
- C1 pad 1: (no net) -> Net-(D2-K)
- C1 pad 2: (no net) -> GND
- C10 pad 1: (no net) -> +3V3
- C10 pad 2: (no net) -> GND
- C11 pad 1: (no net) -> +3V3
- C11 pad 2: (no net) -> GND
- C12 pad 1: (no net) -> VBAT_SENSE
- C12 pad 2: (no net) -> GND
- C13 pad 1: (no net) -> GND
- C13 pad 2: (no net) -> Net-(U8-VRTC)
- C14 pad 1: (no net) -> SIM_BAT
- C14 pad 2: (no net) -> GND
- C15 pad 1: (no net) -> SIM_BAT
- C15 pad 2: (no net) -> GND
- C16 pad 1: (no net) -> FUEL_ADC
- C16 pad 2: (no net) -> GND
- C17 pad 1: (no net) -> /TRACKER/CR1
- C17 pad 2: (no net) -> GND
- C18 pad 1: (no net) -> /TRACKER/CR2
- C18 pad 2: (no net) -> GND
- C19 pad 1: (no net) -> GND
- C19 pad 2: (no net) -> +3V3
- C2 pad 1: (no net) -> Net-(Q1-D)
- C2 pad 2: (no net) -> GND
- C20 pad 1: (no net) -> GND
- C20 pad 2: (no net) -> +3V3
- C21 pad 1: (no net) -> GND
- C21 pad 2: (no net) -> +3V3
- C22 pad 1: (no net) -> GND
- C22 pad 2: (no net) -> +3V3
- C23 pad 1: (no net) -> GND
- C23 pad 2: (no net) -> +3V3
- C24 pad 1: (no net) -> GND
- C24 pad 2: (no net) -> +3V3
- C25 pad 1: (no net) -> GND
- C25 pad 2: (no net) -> +3V3
- C26 pad 1: (no net) -> GND
- C26 pad 2: (no net) -> +3V3
- C27 pad 1: (no net) -> SIM_BAT
- C27 pad 2: (no net) -> GND
- C28 pad 1: (no net) -> GND
- C28 pad 2: (no net) -> +3V3
- C29 pad 1: (no net) -> GND
- C29 pad 2: (no net) -> +3V3
- C30 pad 1: (no net) -> GND
- C30 pad 2: (no net) -> +3V3
- C31 pad 1: (no net) -> GND
- C31 pad 2: (no net) -> +3V3
- C32 pad 1: (no net) -> Net-(U9-C1+)
- C32 pad 2: (no net) -> Net-(U9-C1-)
- C33 pad 1: (no net) -> GND
- C33 pad 2: (no net) -> Net-(U9-VS+)
- C34 pad 1: (no net) -> GND
- C34 pad 2: (no net) -> Net-(U9-VS-)
- C35 pad 1: (no net) -> Net-(U9-C2+)
- C35 pad 2: (no net) -> Net-(U9-C2-)
- C36 pad 1: (no net) -> Net-(U11A-+)
- C36 pad 2: (no net) -> GND
- C37 pad 1: (no net) -> Net-(U13-PC15)
- C37 pad 2: (no net) -> GND
- C38 pad 1: (no net) -> SIM_BAT
- C38 pad 2: (no net) -> GND
- C39 pad 1: (no net) -> SIM_BAT
- C39 pad 2: (no net) -> GND
- C4 pad 1: (no net) -> 5L
- C4 pad 2: (no net) -> GND
- C40 pad 1: (no net) -> Net-(U13-PC14)
- C40 pad 2: (no net) -> GND
- C41 pad 1: (no net) -> GND
- C41 pad 2: (no net) -> Net-(U13-PD0)
- C42 pad 1: (no net) -> GND
- C42 pad 2: (no net) -> Net-(U13-PD1)
- C43 pad 1: (no net) -> GND
- C43 pad 2: (no net) -> +3V3
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Routing:
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- added copper zone on B.Cu, net GND
- added copper zone on F.Cu, net GND
- removed copper zone on B.Cu, net (none)
- removed copper zone on F.Cu, net (none)
